Commit message: sync changes 21.9.20

File: xacros/generated_urdf_from_xacros_here/ovidius_xacro_assembled.urdf (robot description, URDF)
Before this commit: robot ovidius_smm, 5 links, 4 joints
Links:
- added link active_module1, mass 0.892; visual mesh filename=/home/nikos/PhD/projects/Parametric_Simulation_Model_SMM/Ac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 scale=0.001 0.001 0.001
- added link pseudo2b, mass 0.4450127; visual mesh filename=/home/nikos/PhD/projects/Parametric_Simulation_Model_SMM/Ps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 scale=0.001 0.001 0.001
Joints:
- added joint pseudo2a__pseudo2b: type fixed, parent pseudo2a, child pseudo2b, origin xyz=0 0.025 0.118 rpy=1.5708 0 0
- added joint pseudo2b__active_module1: type fixed, parent pseudo2b, child active_module1, origin xyz=0 0.1 0 rpy=0 0 0

File: xacros/ovidius_links_joints_names.xacro (robot description, xacro)
@@ -4,4 +4,6 @@
 <xacro:property name="pseudo_mass_static" value="2.2036439"/>
 <xacro:property name="pseudo_mass_moving" value="0.4450127"/>
+<xacro:property name="active_mass_static" value="0.892"/>
+<xacro:property name="active_mass_moving" value="0.102"/>
 <!-- Pseudo static block-->
 <xacro:macro name="pseudo_static_link_mesh" params="name origin_xyz origin_rpy">
@@ -58,3 +60,49 @@
 </joint>
 </xacro:macro>
+<!-- Fixed assembly parameters-->
+ <xacro:macro name="assembly_active_module2pseudo" params="active_assembly_name  active_assembly_origin_rpy active_assembly_origin_xyz active_assembly_parent active_assembly_child">
+    <joint name="${active_assembly_name}" type="fixed">
+      <origin rpy="${active_assembly_origin_rpy}" xyz="${active_assembly_origin_xyz}" />
+      <parent link="${active_assembly_parent}" />
+      <child link="${active_assembly_child}" />
+    </joint>
+</xacro:macro>
+<!-- Active static block-->
+<xacro:macro name="active_static_link_mesh" params="name origin_xyz origin_rpy">
+    <link name="${name}">
+      <inertial>
+        <origin rpy="0 0 0" xyz="0 0 0"/>
+        <mass value ="${active_mass_static}" />
+        <inertia ixx="0.001" ixy="-1.292e-11" ixz="3.624e-12" iyy="4.195e-04" iyz="-9.613e-06" izz="0.001"/>
+      </inertial>
+      <visual>
+        <origin rpy="${origin_rpy}" xyz="${origin_xyz}" />
+        <geometry>
+          <mesh filename="/home/nikos/PhD/projects/Parametric_Simulation_Model_SMM/Active/active_module_fixed.stl" scale="0.001 0.001 0.001"/>
+        </geometry>
+              <material name="lightgrey">
+        <color rgba="0.95 0.95 0.95 0.5"/>
+      </material>
+      </visual>
+    </link>
+</xacro:macro>
+<!-- Active moving block-->
+<xacro:macro name="active_moving_link_mesh" params="name origin_xyz origin_rpy">
+    <link name="${name}">
+      <inertial>
+        <origin rpy="0 0 0" xyz="0 0 0"/>
+        <mass value ="${active_mass_moving}" />
+        <inertia ixx="3.103e-04" ixy="-3.374e-13" ixz="1.202e-12" iyy="3.187e-04" iyz="8.958e-06" izz="5.995e-05"/>
+      </inertial>
+      <visual>
+        <origin rpy="${origin_rpy}" xyz="${origin_xyz}" />
+        <geometry>
+          <mesh filename="/home/nikos/PhD/projects/Parametric_Simulation_Model_SMM/Active/active_module_moving.stl" scale="0.001 0.001 0.001"/>
+        </geometry>
+        <material name="red">
+          <color rgba="1 0 0 1"/>
+        </material>
+      </visual>
+    </link>
+</xacro:macro>
 </robot>

File: xacros/ovidius_xacro_assembled.xacro (robot description, xacro)
@@ -17,4 +17,16 @@
 <xacro:property name="synthetic2_origin_xyz" value="${synthetic2['synthetic2_origin_xyz']}" />
 <xacro:property name="synthetic2_origin_rpy" value="${synthetic2['synthetic2_origin_rpy']}" />
+<!-- ACTIVE2PSEUDOS FIXED TFs -->
+<xacro:property name="active2pseudo1_yaml_file" value="/home/nikos/PhD/projects/Parametric_Simulation_Model_SMM/yamls/test/active2pseudo_assemblies.yaml" />
+<xacro:property name="active2pseudo1" value="${load_yaml(active2pseudo1_yaml_file)}"/>
+<xacro:property name="active2pseudo1_name" value="${active2pseudo1['active2pseudo1_name']}" />
+<xacro:property name="active2pseudo1_origin_xyz" value="${active2pseudo1['active2pseudo1_origin_xyz']}" />
+<xacro:property name="active2pseudo1_origin_rpy" value="${active2pseudo1['active2pseudo1_origin_rpy']}" />
+<!-- ACTIVE MODULE PARTS -->
+<xacro:property name="active1a_yaml_file" value="/home/nikos/PhD/projects/Parametric_Simulation_Model_SMM/yamls/test/active2pseudo_assemblies.yaml" />
+<xacro:property name="active1a" value="${load_yaml(active1a_yaml_file)}"/>
+<xacro:property name="active1a_name" value="${active1a['active1a_name']}" />
+<xacro:property name="active1a_origin_xyz" value="${active1a['active1a_origin_xyz']}" />
+<xacro:property name="active1a_origin_rpy" value="${active1a['active1a_origin_rpy']}" />
 <!-- PSEUDOJOINTS PARTS -->
 <xacro:property name="pseudo1a_yaml_file" value="/home/nikos/PhD/projects/Parametric_Simulation_Model_SMM/yamls/test/pseudos.yaml" />
@@ -33,4 +45,9 @@
 <xacro:property name="pseudo2a_origin_xyz" value="${pseudo2a['pseudo2a_origin_xyz']}" />
 <xacro:property name="pseudo2a_origin_rpy" value="${pseudo2a['pseudo2a_origin_rpy']}" />
+<xacro:property name="pseudo2b_yaml_file" value="/home/nikos/PhD/projects/Parametric_Simulation_Model_SMM/yamls/test/pseudos.yaml" />
+<xacro:property name="pseudo2b" value="${load_yaml(pseudo2b_yaml_file)}"/>
+<xacro:property name="pseudo2b_name" value="${pseudo2b['pseudo2b_name']}" />
+<xacro:property name="pseudo2b_origin_xyz" value="${pseudo2b['pseudo2b_origin_xyz']}" />
+<xacro:property name="pseudo2b_origin_rpy" value="${pseudo2b['pseudo2b_origin_rpy']}" />
 <!-- PSEUDOJOINTS -->
 <xacro:property name="pseudo1_yaml_file" value="/home/nikos/PhD/projects/Parametric_Simulation_Model_SMM/yamls/test/pseudojoints.yaml" />
@@ -39,4 +56,9 @@
 <xacro:property name="pseudo1_origin_xyz" value="${pseudo1['pseudo1_origin_xyz']}" />
 <xacro:property name="pseudo1_origin_rpy" value="${pseudo1['pseudo1_origin_rpy']}" />
+<xacro:property name="pseudo2_yaml_file" value="/home/nikos/PhD/projects/Parametric_Simulation_Model_SMM/yamls/test/pseudojoints.yaml" />
+<xacro:property name="pseudo2" value="${load_yaml(pseudo2_yaml_file)}"/>
+<xacro:property name="pseudo2_name" value="${pseudo2['pseudo1_name']}" />
+<xacro:property name="pseudo2_origin_xyz" value="${pseudo1['pseudo2_origin_xyz']}" />
+<xacro:property name="pseudo2_origin_rpy" value="${pseudo1['pseudo2_origin_rpy']}" />
 <!-- END - Include -->
 <!-- ROBOT DESCRIPTION-->
@@ -75,6 +97,14 @@
 <xacro:pseudo_moving_link_mesh name="${pseudo1b_name}" origin_xyz="${pseudo1b_origin_xyz}" origin_rpy="${pseudo1b_origin_rpy}"/>
 <!-- This joint is parameterized for SJ2:C011-->
-<xacro:synthetic_joint_name  synthetic_name="${pseudo1b_name}__pseudo2a"  synthetic_origin_rpy="${synthetic2_origin_rpy}" synthetic_origin_xyz="${synthetic2_origin_xyz}" synthetic_parent="${pseudo1b_name}" synthetic_child="${pseudo2a_name}" />
+<xacro:synthetic_joint_name  synthetic_name="${pseudo1b_name}__${pseudo2a_name}"  synthetic_origin_rpy="${synthetic2_origin_rpy}" synthetic_origin_xyz="${synthetic2_origin_xyz}" synthetic_parent="${pseudo1b_name}" synthetic_child="${pseudo2a_name}" />
 <!-- Start building Pseudojoint 2 STATIC PART-->
 <xacro:pseudo_static_link_mesh name="${pseudo2a_name}" origin_xyz="${pseudo2a_origin_xyz}" origin_rpy="${pseudo2a_origin_rpy}"/>
+<!-- PSEUDO2 CONFIGURATION -->
+<xacro:pseudo_joint_name  pseudo_name="${pseudo2a_name}__${pseudo2b_name}"  pseudo_origin_rpy="${pseudo2_origin_rpy}" pseudo_origin_xyz="${pseudo2_origin_xyz}" pseudo_parent="${pseudo2a_name}" pseudo_child="${pseudo2b_name}" />
+<!-- Start building Pseudojoint 2 MOVING PART-->
+<xacro:pseudo_moving_link_mesh name="${pseudo2b_name}" origin_xyz="${pseudo2b_origin_xyz}" origin_rpy="${pseudo2b_origin_rpy}"/>
+<!-- This fixed tf assembles active module of link to preceding pseudo-->
+<xacro:assembly_active_module2pseudo  active_assembly_name="${pseudo2b_name}__${active1a_name}"  active_assembly_origin_rpy="${active2pseudo1_origin_rpy}" active_assembly_origin_xyz="${active2pseudo1_origin_xyz}" active_assembly_parent="${pseudo2b_name}" active_assembly_child="${active1a_name}" />
+<!-- Adds Active Module MOVING PART-->
+<xacro:active_static_link_mesh name="${active1a_name}" origin_xyz="${active1a_origin_xyz}" origin_rpy="${active1a_origin_rpy}"/>
 </robot>
