Commit message: sync changes 22.9.20

File: xacros/generated_urdf_from_xacros_here/ovidius_xacro_assembled.urdf (robot description, URDF)
Before this commit: robot ovidius_smm, 7 links, 6 joints
Links:
- removed link active_module1
- added link active_module1a, mass 0.892; visual mesh filename=/home/nikos/PhD/projects/Parametric_Simulation_Model_SMM/Ac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 scale=0.001 0.001 0.001
- added link active_module1b, mass 0.102; visual mesh filename=/home/nikos/PhD/projects/Parametric_Simulation_Model_SMM/Ac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 scale=0.001 0.001 0.001
- added link pseudo3a, mass 2.2036439; visual mesh filename=/home/nikos/PhD/projects/Parametric_Simulation_Model_SMM/Ps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 scale=0.001 0.001 0.001
- added link pseudo3b, mass 0.4450127; visual mesh filename=/home/nikos/PhD/projects/Parametric_Simulation_Model_SMM/Ps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 scale=0.001 0.001 0.001
- added link pseudo4a, mass 2.2036439; visual mesh filename=/home/nikos/PhD/projects/Parametric_Simulation_Model_SMM/Ps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 scale=0.001 0.001 0.001
- added link pseudo4b, mass 0.4450127; visual mesh filename=/home/nikos/PhD/projects/Parametric_Simulation_Model_SMM/Ps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 scale=0.001 0.001 0.001
Joints:
- removed joint pseudo2b__active_module1
- added joint active_module1a__active_module1b: type revolute, parent active_module1a, child active_module1b, origin xyz=0 0.032 0 rpy=0 0 0, axis 0 0 1, limit lower=-2 upper=2 effort=55 velocity=4.0841
- added joint active_module1b__pseudo3a: type fixed, parent active_module1b, child pseudo3a, origin xyz=0 0.0955 -0.05 rpy=0 0 0
- added joint pseudo2b__active_module1a: type fixed, parent pseudo2b, child active_module1a, origin xyz=0 0.1 0 rpy=0 1.5708 0
- added joint pseudo3a__pseudo3b: type fixed, parent pseudo3a, child pseudo3b, origin xyz=0 0.025 0.118 rpy=1.5708 0 0
- added joint pseudo3b__pseudo4a: type fixed, parent pseudo3b, child pseudo4a, origin xyz=-0.075 0.1444 0 rpy=0 1.5708 0
- added joint pseudo4a__pseudo4b: type fixed, parent pseudo4a, child pseudo4b, origin xyz=0 0.025 0.118 rpy=1.5708 0 0

File: xacros/ovidius_links_joints_names.xacro (robot description, xacro)
@@ -100,9 +100,20 @@
           <mesh filename="/home/nikos/PhD/projects/Parametric_Simulation_Model_SMM/Active/active_module_moving.stl" scale="0.001 0.001 0.001"/>
         </geometry>
-        <material name="red">
-          <color rgba="1 0 0 1"/>
+        <material name="black">
+          <color rgba="0.1 0.1 0.1 1"/>
         </material>
       </visual>
     </link>
 </xacro:macro>
+<!-- Synthetic joint parameters-->
+ <xacro:macro name="dxlPROp_joint" params="active_name  active_origin_rpy active_origin_xyz active_parent active_child">
+    <joint name="${active_name}" type="revolute">
+      <origin rpy="${active_origin_rpy}" xyz="${active_origin_xyz}" />
+      <parent link="${active_parent}" />
+      <child link="${active_child}" />
+      <axis xyz="0 0 1"/>
+      <limit effort="55" lower="-2" upper="2" velocity="4.0841"/>
+      <dynamics damping="0.5"/>
+    </joint>
+</xacro:macro>
 </robot>

File: xacros/ovidius_xacro_assembled.xacro (robot description, xacro)
@@ -7,58 +7,94 @@
 <!-- INCLUDE YAML PROPERTIES FILES FOR EACH STRUCTURE BUILDING BLOCK-->
 <!-- SYNTHETIC JOINTS -->
-<xacro:property name="synthetic1_yaml_file" value="/home/nikos/PhD/projects/Parametric_Simulation_Model_SMM/yamls/test/synthetics.yaml" />
-<xacro:property name="synthetic1" value="${load_yaml(synthetic1_yaml_file)}"/>
+<xacro:property name="synthetics_properties_definition_file" value="/home/nikos/PhD/projects/Parametric_Simulation_Model_SMM/yamls/test/synthetics.yaml" />
+<xacro:property name="synthetic1" value="${load_yaml(synthetics_properties_definition_file)}"/>
 <xacro:property name="synthetic1_name" value="${synthetic1['synthetic1_name']}" />
 <xacro:property name="synthetic1_origin_xyz" value="${synthetic1['synthetic1_origin_xyz']}" />
 <xacro:property name="synthetic1_origin_rpy" value="${synthetic1['synthetic1_origin_rpy']}" />
-<xacro:property name="synthetic2_yaml_file" value="/home/nikos/PhD/projects/Parametric_Simulation_Model_SMM/yamls/test/synthetics.yaml" />
-<xacro:property name="synthetic2" value="${load_yaml(synthetic2_yaml_file)}"/>
+<xacro:property name="synthetic2" value="${load_yaml(synthetics_properties_definition_file)}"/>
 <xacro:property name="synthetic2_name" value="${synthetic2['synthetic2_name']}" />
 <xacro:property name="synthetic2_origin_xyz" value="${synthetic2['synthetic2_origin_xyz']}" />
 <xacro:property name="synthetic2_origin_rpy" value="${synthetic2['synthetic2_origin_rpy']}" />
+<xacro:property name="synthetic3" value="${load_yaml(synthetics_properties_definition_file)}"/>
+<xacro:property name="synthetic3_name" value="${synthetic3['synthetic3_name']}" />
+<xacro:property name="synthetic3_origin_xyz" value="${synthetic3['synthetic3_origin_xyz']}" />
+<xacro:property name="synthetic3_origin_rpy" value="${synthetic3['synthetic3_origin_rpy']}" />
+<xacro:property name="synthetic4" value="${load_yaml(synthetics_properties_definition_file)}"/>
+<xacro:property name="synthetic4_name" value="${synthetic4['synthetic4_name']}" />
+<xacro:property name="synthetic4_origin_xyz" value="${synthetic4['synthetic4_origin_xyz']}" />
+<xacro:property name="synthetic4_origin_rpy" value="${synthetic4['synthetic4_origin_rpy']}" />
 <!-- ACTIVE2PSEUDOS FIXED TFs -->
-<xacro:property name="active2pseudo1_yaml_file" value="/home/nikos/PhD/projects/Parametric_Simulation_Model_SMM/yamls/test/active2pseudo_assemblies.yaml" />
-<xacro:property name="active2pseudo1" value="${load_yaml(active2pseudo1_yaml_file)}"/>
+<xacro:property name="active2pseudojoints_configuration_file" value="/home/nikos/PhD/projects/Parametric_Simulation_Model_SMM/yamls/test/active2pseudo_assemblies.yaml" />
+<xacro:property name="active2pseudo1" value="${load_yaml(active2pseudojoints_configuration_file)}"/>
 <xacro:property name="active2pseudo1_name" value="${active2pseudo1['active2pseudo1_name']}" />
 <xacro:property name="active2pseudo1_origin_xyz" value="${active2pseudo1['active2pseudo1_origin_xyz']}" />
 <xacro:property name="active2pseudo1_origin_rpy" value="${active2pseudo1['active2pseudo1_origin_rpy']}" />
 <!-- ACTIVE MODULE PARTS -->
-<xacro:property name="active1a_yaml_file" value="/home/nikos/PhD/projects/Parametric_Simulation_Model_SMM/yamls/test/active2pseudo_assemblies.yaml" />
-<xacro:property name="active1a" value="${load_yaml(active1a_yaml_file)}"/>
+<xacro:property name="active_properties_definition_file" value="/home/nikos/PhD/projects/Parametric_Simulation_Model_SMM/yamls/test/active2pseudo_assemblies.yaml" />
+<xacro:property name="active1a" value="${load_yaml(active_properties_definition_file)}"/>
 <xacro:property name="active1a_name" value="${active1a['active1a_name']}" />
 <xacro:property name="active1a_origin_xyz" value="${active1a['active1a_origin_xyz']}" />
 <xacro:property name="active1a_origin_rpy" value="${active1a['active1a_origin_rpy']}" />
+<xacro:property name="active1b" value="${load_yaml(active_properties_definition_file)}"/>
+<xacro:property name="active1b_name" value="${active1b['active1b_name']}" />
+<xacro:property name="active1b_origin_xyz" value="${active1b['active1b_origin_xyz']}" />
+<xacro:property name="active1b_origin_rpy" value="${active1b['active1b_origin_rpy']}" />
+<!-- ACTIVE JOINTS -->
+<xacro:property name="active1" value="${load_yaml(active_properties_definition_file)}"/>
+<xacro:property name="active1_name" value="${active1['active1_name']}" />
+<xacro:property name="active1_origin_xyz" value="${active1['active1_origin_xyz']}" />
+<xacro:property name="active1_origin_rpy" value="${active1['active1_origin_rpy']}" />
 <!-- PSEUDOJOINTS PARTS -->
-<xacro:property name="pseudo1a_yaml_file" value="/home/nikos/PhD/projects/Parametric_Simulation_Model_SMM/yamls/test/pseudos.yaml" />
-<xacro:property name="pseudo1a" value="${load_yaml(pseudo1a_yaml_file)}"/>
+<xacro:property name="pseudo_modules_properties_definition_file" value="/home/nikos/PhD/projects/Parametric_Simulation_Model_SMM/yamls/test/pseudos.yaml" />
+<xacro:property name="pseudo1a" value="${load_yaml(pseudo_modules_properties_definition_file)}"/>
 <xacro:property name="pseudo1a_name" value="${pseudo1a['pseudo1a_name']}" />
 <xacro:property name="pseudo1a_origin_xyz" value="${pseudo1a['pseudo1a_origin_xyz']}" />
 <xacro:property name="pseudo1a_origin_rpy" value="${pseudo1a['pseudo1a_origin_rpy']}" />
-<xacro:property name="pseudo1b_yaml_file" value="/home/nikos/PhD/projects/Parametric_Simulation_Model_SMM/yamls/test/pseudos.yaml" />
-<xacro:property name="pseudo1b" value="${load_yaml(pseudo1b_yaml_file)}"/>
+<xacro:property name="pseudo1b" value="${load_yaml(pseudo_modules_properties_definition_file)}"/>
 <xacro:property name="pseudo1b_name" value="${pseudo1b['pseudo1b_name']}" />
 <xacro:property name="pseudo1b_origin_xyz" value="${pseudo1b['pseudo1b_origin_xyz']}" />
 <xacro:property name="pseudo1b_origin_rpy" value="${pseudo1b['pseudo1b_origin_rpy']}" />
-<xacro:property name="pseudo2a_yaml_file" value="/home/nikos/PhD/projects/Parametric_Simulation_Model_SMM/yamls/test/pseudos.yaml" />
-<xacro:property name="pseudo2a" value="${load_yaml(pseudo2a_yaml_file)}"/>
+<xacro:property name="pseudo2a" value="${load_yaml(pseudo_modules_properties_definition_file)}"/>
 <xacro:property name="pseudo2a_name" value="${pseudo2a['pseudo2a_name']}" />
 <xacro:property name="pseudo2a_origin_xyz" value="${pseudo2a['pseudo2a_origin_xyz']}" />
 <xacro:property name="pseudo2a_origin_rpy" value="${pseudo2a['pseudo2a_origin_rpy']}" />
-<xacro:property name="pseudo2b_yaml_file" value="/home/nikos/PhD/projects/Parametric_Simulation_Model_SMM/yamls/test/pseudos.yaml" />
-<xacro:property name="pseudo2b" value="${load_yaml(pseudo2b_yaml_file)}"/>
+<xacro:property name="pseudo2b" value="${load_yaml(pseudo_modules_properties_definition_file)}"/>
 <xacro:property name="pseudo2b_name" value="${pseudo2b['pseudo2b_name']}" />
 <xacro:property name="pseudo2b_origin_xyz" value="${pseudo2b['pseudo2b_origin_xyz']}" />
 <xacro:property name="pseudo2b_origin_rpy" value="${pseudo2b['pseudo2b_origin_rpy']}" />
+<xacro:property name="pseudo3a" value="${load_yaml(pseudo_modules_properties_definition_file)}"/>
+<xacro:property name="pseudo3a_name" value="${pseudo3a['pseudo3a_name']}" />
+<xacro:property name="pseudo3a_origin_xyz" value="${pseudo3a['pseudo3a_origin_xyz']}" />
+<xacro:property name="pseudo3a_origin_rpy" value="${pseudo3a['pseudo3a_origin_rpy']}" />
+<xacro:property name="pseudo3b" value="${load_yaml(pseudo_modules_properties_definition_file)}"/>
+<xacro:property name="pseudo3b_name" value="${pseudo3b['pseudo3b_name']}" />
+<xacro:property name="pseudo3b_origin_xyz" value="${pseudo3b['pseudo3b_origin_xyz']}" />
+<xacro:property name="pseudo3b_origin_rpy" value="${pseudo3b['pseudo3b_origin_rpy']}" />
+<xacro:property name="pseudo4a" value="${load_yaml(pseudo_modules_properties_definition_file)}"/>
+<xacro:property name="pseudo4a_name" value="${pseudo3a['pseudo4a_name']}" />
+<xacro:property name="pseudo4a_origin_xyz" value="${pseudo4a['pseudo4a_origin_xyz']}" />
+<xacro:property name="pseudo4a_origin_rpy" value="${pseudo4a['pseudo4a_origin_rpy']}" />
+<xacro:property name="pseudo4b" value="${load_yaml(pseudo_modules_properties_definition_file)}"/>
+<xacro:property name="pseudo4b_name" value="${pseudo4b['pseudo4b_name']}" />
+<xacro:property name="pseudo4b_origin_xyz" value="${pseudo4b['pseudo4b_origin_xyz']}" />
+<xacro:property name="pseudo4b_origin_rpy" value="${pseudo4b['pseudo4b_origin_rpy']}" />
 <!-- PSEUDOJOINTS -->
-<xacro:property name="pseudo1_yaml_file" value="/home/nikos/PhD/projects/Parametric_Simulation_Model_SMM/yamls/test/pseudojoints.yaml" />
-<xacro:property name="pseudo1" value="${load_yaml(pseudo1_yaml_file)}"/>
+<xacro:property name="pseudojoints_configuration_file" value="/home/nikos/PhD/projects/Parametric_Simulation_Model_SMM/yamls/test/pseudojoints.yaml" />
+<xacro:property name="pseudo1" value="${load_yaml(pseudojoints_configuration_file)}"/>
 <xacro:property name="pseudo1_name" value="${pseudo1['pseudo1_name']}" />
 <xacro:property name="pseudo1_origin_xyz" value="${pseudo1['pseudo1_origin_xyz']}" />
 <xacro:property name="pseudo1_origin_rpy" value="${pseudo1['pseudo1_origin_rpy']}" />
-<xacro:property name="pseudo2_yaml_file" value="/home/nikos/PhD/projects/Parametric_Simulation_Model_SMM/yamls/test/pseudojoints.yaml" />
-<xacro:property name="pseudo2" value="${load_yaml(pseudo2_yaml_file)}"/>
+<xacro:property name="pseudo2" value="${load_yaml(pseudojoints_configuration_file)}"/>
 <xacro:property name="pseudo2_name" value="${pseudo2['pseudo1_name']}" />
-<xacro:property name="pseudo2_origin_xyz" value="${pseudo1['pseudo2_origin_xyz']}" />
-<xacro:property name="pseudo2_origin_rpy" value="${pseudo1['pseudo2_origin_rpy']}" />
+<xacro:property name="pseudo2_origin_xyz" value="${pseudo2['pseudo2_origin_xyz']}" />
+<xacro:property name="pseudo2_origin_rpy" value="${pseudo2['pseudo2_origin_rpy']}" />
+<xacro:property name="pseudo3" value="${load_yaml(pseudojoints_configuration_file)}"/>
+<xacro:property name="pseudo3_name" value="${pseudo3['pseudo3_name']}" />
+<xacro:property name="pseudo3_origin_xyz" value="${pseudo3['pseudo3_origin_xyz']}" />
+<xacro:property name="pseudo3_origin_rpy" value="${pseudo3['pseudo3_origin_rpy']}" />
+<xacro:property name="pseudo4" value="${load_yaml(pseudojoints_configuration_file)}"/>
+<xacro:property name="pseudo4_name" value="${pseudo4['pseudo4_name']}" />
+<xacro:property name="pseudo4_origin_xyz" value="${pseudo4['pseudo4_origin_xyz']}" />
+<xacro:property name="pseudo4_origin_rpy" value="${pseudo4['pseudo4_origin_rpy']}" />
 <!-- END - Include -->
 <!-- ROBOT DESCRIPTION-->
@@ -106,5 +142,25 @@
 <!-- This fixed tf assembles active module of link to preceding pseudo-->
 <xacro:assembly_active_module2pseudo  active_assembly_name="${pseudo2b_name}__${active1a_name}"  active_assembly_origin_rpy="${active2pseudo1_origin_rpy}" active_assembly_origin_xyz="${active2pseudo1_origin_xyz}" active_assembly_parent="${pseudo2b_name}" active_assembly_child="${active1a_name}" />
+<!-- Adds Active Module STATIC PART-->
+<xacro:active_static_link_mesh name="${active1a_name}" origin_xyz="${active1a_origin_xyz}" origin_rpy="${active1a_origin_rpy}"/>
+<!-- Adds DXL Active joint -->
+<xacro:dxlPROp_joint active_name="${active1a_name}__${active1b_name}"  active_origin_rpy="${active1_origin_rpy}" active_origin_xyz="${active1_origin_xyz}" active_parent="${active1a_name}" active_child="${active1b_name}"/>
 <!-- Adds Active Module MOVING PART-->
-<xacro:active_static_link_mesh name="${active1a_name}" origin_xyz="${active1a_origin_xyz}" origin_rpy="${active1a_origin_rpy}"/>
+<xacro:active_moving_link_mesh name="${active1b_name}" origin_xyz="${active1b_origin_xyz}" origin_rpy="${active1b_origin_rpy}"/>
+<!-- This joint is parameterized for SJ3:C01101 -->
+<xacro:synthetic_joint_name  synthetic_name="${active1b_name}__${pseudo3a_name}"  synthetic_origin_rpy="${synthetic3_origin_rpy}" synthetic_origin_xyz="${synthetic3_origin_xyz}" synthetic_parent="${active1b_name}" synthetic_child="${pseudo3a_name}" />
+<!-- Start building Pseudojoint 3 STATIC PART-->
+<xacro:pseudo_static_link_mesh name="${pseudo3a_name}" origin_xyz="${pseudo3a_origin_xyz}" origin_rpy="${pseudo3a_origin_rpy}"/>
+<!-- PSEUDO3 CONFIGURATION -->
+<xacro:pseudo_joint_name  pseudo_name="${pseudo3a_name}__${pseudo3b_name}"  pseudo_origin_rpy="${pseudo3_origin_rpy}" pseudo_origin_xyz="${pseudo3_origin_xyz}" pseudo_parent="${pseudo3a_name}" pseudo_child="${pseudo3b_name}" />
+<!-- Start building Pseudojoint 3 MOVING PART-->
+<xacro:pseudo_moving_link_mesh name="${pseudo3b_name}" origin_xyz="${pseudo3b_origin_xyz}" origin_rpy="${pseudo3b_origin_rpy}"/>
+<!-- This joint is parameterized for SJ4:C011011-->
+<xacro:synthetic_joint_name  synthetic_name="${pseudo3b_name}__${pseudo4a_name}"  synthetic_origin_rpy="${synthetic4_origin_rpy}" synthetic_origin_xyz="${synthetic4_origin_xyz}" synthetic_parent="${pseudo3b_name}" synthetic_child="${pseudo4a_name}" />
+<!-- Start building Pseudojoint 4 STATIC PART-->
+<xacro:pseudo_static_link_mesh name="${pseudo4a_name}" origin_xyz="${pseudo4a_origin_xyz}" origin_rpy="${pseudo4a_origin_rpy}"/>
+<!-- PSEUDO4 CONFIGURATION -->
+<xacro:pseudo_joint_name  pseudo_name="${pseudo4a_name}__${pseudo4b_name}"  pseudo_origin_rpy="${pseudo4_origin_rpy}" pseudo_origin_xyz="${pseudo4_origin_xyz}" pseudo_parent="${pseudo4a_name}" pseudo_child="${pseudo4b_name}" />
+<!-- Start building Pseudojoint 4 MOVING PART-->
+<xacro:pseudo_moving_link_mesh name="${pseudo4b_name}" origin_xyz="${pseudo4b_origin_xyz}" origin_rpy="${pseudo4b_origin_rpy}"/>
 </robot>

Commit message: finished simple xacro assembly file for S0110110 structure, defined all structural blocks

File: xacros/generated_urdf_from_xacros_here/ovidius_xacro_assembled.urdf (robot description, URDF)
Before this commit: robot ovidius_smm, 12 links, 11 joints
Links:
- added link active_module2a, mass 0.892; visual mesh filename=/home/nikos/PhD/projects/Parametric_Simulation_Model_SMM/Ac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 scale=0.001 0.001 0.001
- added link active_module2b, mass 0.102; visual mesh filename=/home/nikos/PhD/projects/Parametric_Simulation_Model_SMM/Ac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 scale=0.001 0.001 0.001
Joints:
- added joint active_module2a__active_module2b: type revolute, parent active_module2a, child active_module2b, origin xyz=0 0.032 0 rpy=0 0 0, axis 0 0 1, limit lower=-2 upper=2 effort=55 velocity=4.0841
- added joint pseudo4b__active_module2a: type fixed, parent pseudo4b, child active_module2a, origin xyz=0 0.1 0 rpy=0 1.5708 0

File: xacros/ovidius_links_joints_names.xacro (robot description, xacro)
@@ -1,4 +1,5 @@
 <?xml version="1.0" ?>
 <robot xmlns:xacro="http://www.ros.org/wiki/xacro">
+<!-- ALL components used to assemble the Ovidius SMM are defined here. This file should be xacro:included in each xacro:assembly robot urdf file! -->
 <!-- MASS parameters for Pseudojoint Design-->
 <xacro:property name="pseudo_mass_static" value="2.2036439"/>
@@ -81,6 +82,6 @@
           <mesh filename="/home/nikos/PhD/projects/Parametric_Simulation_Model_SMM/Active/active_module_fixed.stl" scale="0.001 0.001 0.001"/>
         </geometry>
-              <material name="lightgrey">
-        <color rgba="0.95 0.95 0.95 0.5"/>
+              <material name="lightblack">
+        <color rgba="0.25 0.25 0.25 0.25"/>
       </material>
       </visual>
