Commit message: Started conditioned parametric structure assembly

File: xacros/conditioned_parameterized_SMM_assembly.xacro (robot description, xacro)
@@ -5,5 +5,29 @@
 <!-- I.1.	INCLUDE XACROS THAT CONTAIN STRUCTURE BUILDING BLOCKS-->
 <xacro:include filename="/home/nikos/PhD/projects/Parametric_Simulation_Model_SMM/xacros/ovidius_links_joints_names.xacro" />
-<!-- I.2	INCLUDE YAML PROPERTIES FILES FOR EACH STRUCTURE BUILDING BLOCK-->
+<!-- I.2	INCLUDE YAML PROPERTIES FILE FOR EACH STRUCTURE BUILDING BLOCK-->
+<xacro:property name="definitions_file" value="/home/nikos/PhD/projects/Parametric_Simulation_Model_SMM/yamls/test/tf_list_for_conditioned_assembly.yaml" />
+<!-- SYNTHETIC JOINTS -->
+<xacro:property name="synthetic1" value="${load_yaml(definitions_file)}"/>
+<xacro:property name="synthetic1_name" value="${synthetic1['synthetic1_name']}" />
+<xacro:property name="synthetic1_origin_xyz" value="${synthetic1['synthetic1_origin_xyz']}" />
+<xacro:property name="synthetic1_origin_rpy" value="${synthetic1['synthetic1_origin_rpy']}" />
+<!-- PSEUDOJOINTS PARTS -->
+<xacro:property name="pseudo1a" value="${load_yaml(definitions_file)}"/>
+<xacro:property name="pseudo1a_name" value="${pseudo1a['pseudo_a_name']}" />
+<xacro:property name="pseudo1a_origin_xyz" value="${pseudo1a['pseudo_a_origin_xyz']}" />
+<xacro:property name="pseudo1a_origin_rpy" value="${pseudo1a['pseudo_a_origin_rpy']}" />
+<xacro:property name="pseudo1b" value="${load_yaml(definitions_file)}"/>
+<xacro:property name="pseudo1b_name" value="${pseudo1b['pseudo_b_name']}" />
+<xacro:property name="pseudo1b_origin_xyz" value="${pseudo1b['pseudo_b_origin_xyz']}" />
+<xacro:property name="pseudo1b_origin_rpy" value="${pseudo1b['pseudo_b_origin_rpy']}" />
+<!-- PSEUDOJOINTS -->
+<xacro:property name="pseudo1" value="${load_yaml(definitions_file)}"/>
+<xacro:property name="pseudo1_name" value="${pseudo1['pseudo_name']}" />
+<xacro:property name="pseudo1_origin_xyz" value="${pseudo1['pseudo_origin_xyz']}" />
+<xacro:property name="pseudo1_origin_r" value="${pseudo1['pseudo_origin_r']}" />
+<xacro:property name="pseudo1_origin_p" value="${pseudo1['pseudo_origin_p']}" />
+<xacro:property name="pseudo1_origin_y" value="${pseudo1['pseudo_origin_y']}" />
+<!-- PSEUDOJOINTS' ANGLES: USER SPECIFIED!!! this values should be added to the Rx compartment of rotation values-->
+<xacro:property name="pseudo1_angle" value="1"/>
 <!-- II.1	STRUCTURE STRING DEFINITION. This is imported by user  in the yaml file, based on desired structure/optimization results-->
 <xacro:property name="structure_string_definitions" value="/home/nikos/PhD/projects/Parametric_Simulation_Model_SMM/yamls/test/test_structure_string_definition.yaml" />
@@ -17,3 +41,43 @@
 <xacro:property name="s7" value="${string_elements['s7']}" />
 <!-- III.1	ROBOT to be generated to URDF model-->
+<!-- ROBOT DESCRIPTION-->
+<link name="world"/>
+<!-- S -0- This is first revolute joint -->
+<joint name="world__base_link" type="revolute">
+<origin rpy="0 0 0" xyz="0 0 0"/>
+<parent link="world"/>
+<child link="base_link"/>
+<axis xyz="0 0 1"/>
+<limit effort="55" lower="-2" upper="2" velocity="4.0841"/>
+<dynamics damping="0.5"/>
+</joint>
+<!-- METAMORPHIC LINK 1: BODY "base_link" AND the first pseudo are ALWAYS fixed-->
+<link name="base_link">
+    <inertial>
+      <origin rpy="0 0 0" xyz="0.00205 0.00373 0.020774"/>
+      <mass value ="0.500" />
+      <inertia ixx="5.063e-004" ixy="2.773e-005" ixz="7.042e-007" iyy="5.387e-004" iyz="1.237e-006" izz="7.207e-004"/>
+    </inertial>
+    <visual>
+      <origin rpy="0 0 0.5" xyz="0 0 0"/>
+      <geometry>
+        <mesh filename="/home/nikos/PhD/projects/Parametric_Simulation_Model_SMM/baselink/ovidius_smm_baselink.stl" scale="0.001 0.001 0.001"/>
+      </geometry>
+      <material name="gray">
+        <color rgba="0.5 0.5 0.5 0.9"/>
+      </material>
+    </visual>
+</link>
+<!-- HERE checks conditions for 1st metamorphic link-->
+<xacro:unless value="${s2 == 9}"> <!-- if pseudo in this position of structure chain exists continue checking for assembly details -->
+  	<xacro:if value="${s2 == 21}">
+ 		<xacro:synthetic_joint_name  synthetic_name="base_link__${pseudo1a_name}"  synthetic_origin_rpy="${synthetic1_origin_rpy}" synthetic_origin_xyz="${synthetic1_origin_xyz}" synthetic_parent="base_link" synthetic_child="${pseudo1a_name}" />
+		<!-- Start building Pseudojoint 1 STATIC PART-->
+		<xacro:pseudo_static_link_mesh name="${pseudo1a_name}" origin_xyz="${pseudo1a_origin_xyz}" origin_rpy="${pseudo1a_origin_rpy}"/>
+		<!-- PSEUDO1 CONFIGURATION -->
+		<xacro:pseudo_joint_name  pseudo_name="${pseudo1a_name}__${pseudo1b_name}"  pseudo_origin_rpy="${pseudo1_origin_r+pseudo1_angle} ${pseudo1_origin_p} ${pseudo1_origin_y}" pseudo_origin_xyz="${pseudo1_origin_xyz}" pseudo_parent="${pseudo1a_name}" pseudo_child="${pseudo1b_name}" />
+		<!-- Start building Pseudojoint 1 MOVING PART-->
+		<xacro:pseudo_moving_link_mesh name="${pseudo1b_name}" origin_xyz="${pseudo1b_origin_xyz}" origin_rpy="${pseudo1b_origin_rpy}"/>
+	</xacro:if>
+</xacro:unless>
 </robot>
