Commit message: Updated conditioned parametric structure assembly 23.9.20

File: xacros/conditioned_parameterized_SMM_assembly.xacro (robot description, xacro)
@@ -201,23 +201,141 @@
 </xacro:if>
 <!-- STARTED SECOND METAMORPHIC LINK -->
-<xacro:unless value="${s5 == 9}"> <!-- if pseudo in this position of structure chain exists continue checking for assembly details -->
-			<xacro:if value="${s5 == 31}">
-				<xacro:synthetic_joint_name  synthetic_name="${active_b_name}_${active_cnt}__${pseudo_a_name}_3"  synthetic_origin_rpy="${synthetic3_origin_r} ${synthetic3_origin_p} ${synthetic3_origin_ry}" synthetic_origin_xyz="${synthetic3_origin_x} ${synthetic3_origin_y} ${synthetic3_origin_z}" synthetic_parent="${active_b_name}_1" synthetic_child="${pseudo_a_name}_3" />
-				<!-- Start building Pseudojoint 3 STATIC PART-->
-				<xacro:pseudo_static_link_mesh name="${pseudo_a_name}_3" origin_xyz="${pseudo_a_origin_xyz}" origin_rpy="${pseudo_a_origin_rpy}"/>
+<xacro:unless value="${s5 == 9}"> <!--  First case is this meta link had pseudo in first string parameter-->
+	<xacro:unless value="${s2 == 9 or s3==9}"> <!--  First sub-case is previous meta link had 2 pseudos-->
+		<xacro:property name="last_pseudo_cnt" value="2" />
+		<xacro:property name="pseudo_cnt" value="3" />
+		<xacro:if value="${s5 == 31}">
+			<xacro:synthetic_joint_name  synthetic_name="${active_b_name}_${active_cnt}__${pseudo_a_name}_${pseudo_cnt}"  synthetic_origin_rpy="${synthetic3_origin_r} ${synthetic3_origin_p} ${synthetic3_origin_ry}" synthetic_origin_xyz="${synthetic3_origin_x} ${synthetic3_origin_y} ${synthetic3_origin_z}" synthetic_parent="${active_b_name}_${active_cnt}" synthetic_child="${pseudo_a_name}_${pseudo_cnt}" />
+			<!-- Start building Pseudojoint 3 STATIC PART-->
+			<xacro:pseudo_static_link_mesh name="${pseudo_a_name}_${pseudo_cnt}" origin_xyz="${pseudo_a_origin_xyz}" origin_rpy="${pseudo_a_origin_rpy}"/>
+			<!-- PSEUDO2 CONFIGURATION -->
+			<xacro:pseudo_joint_name  pseudo_name="${pseudo_a_name}_${pseudo_cnt}__${pseudo_b_name}_${pseudo_cnt}"  pseudo_origin_rpy="${pseudo_origin_r+pseudo3_angle} ${pseudo_origin_p} ${pseudo_origin_y}" pseudo_origin_xyz="${pseudo_origin_xyz}" pseudo_parent="${pseudo_a_name}_${pseudo_cnt}" pseudo_child="${pseudo_b_name}_${pseudo_cnt}" />
+			<!-- Start building Pseudojoint 3 MOVING PART-->
+			<xacro:pseudo_moving_link_mesh name="${pseudo_b_name}_${pseudo_cnt}" origin_xyz="${pseudo_b_origin_xyz}" origin_rpy="${pseudo_b_origin_rpy}"/>
+		</xacro:if>
+		<xacro:if value="${s5 == 21}">
+			<xacro:synthetic_joint_name  synthetic_name="${active_b_name}_${active_cnt}__${pseudo_a_name}_${pseudo_cnt}"  synthetic_origin_rpy="${synthetic5_origin_r} ${synthetic5_origin_p} ${synthetic5_origin_ry}" synthetic_origin_xyz="${synthetic5_origin_x} ${synthetic5_origin_y} ${synthetic5_origin_z}" synthetic_parent="${active_b_name}_${active_cnt}" synthetic_child="${pseudo_a_name}_${pseudo_cnt}" />
+			<!-- Start building Pseudojoint 3 STATIC PART-->
+			<xacro:pseudo_static_link_mesh name="${pseudo_a_name}_${pseudo_cnt}" origin_xyz="${pseudo_a_origin_xyz}" origin_rpy="${pseudo_a_origin_rpy}"/>
+			<!-- PSEUDO2 CONFIGURATION -->
+			<xacro:pseudo_joint_name  pseudo_name="${pseudo_a_name}_${pseudo_cnt}__${pseudo_b_name}_${pseudo_cnt}"  pseudo_origin_rpy="${pseudo_origin_r+pseudo3_angle} ${pseudo_origin_p} ${pseudo_origin_y}" pseudo_origin_xyz="${pseudo_origin_xyz}" pseudo_parent="${pseudo_a_name}_${pseudo_cnt}" pseudo_child="${pseudo_b_name}_${pseudo_cnt}" />
+			<!-- Start building Pseudojoint 3 MOVING PART-->
+			<xacro:pseudo_moving_link_mesh name="${pseudo_b_name}_${pseudo_cnt}" origin_xyz="${pseudo_b_origin_xyz}" origin_rpy="${pseudo_b_origin_rpy}"/>
+		</xacro:if>
+		<!-- Now evaluate next string of meta link!-->
+		<xacro:unless value="${s6 == 9}">
+			<xacro:property name="last_pseudo_cnt" value="3" />
+			<xacro:property name="pseudo_cnt" value="4" />
+			<xacro:if value="${s6 == 21}">
+				<xacro:synthetic_joint_name  synthetic_name="${pseudo_b_name}_${last_pseudo_cnt}__${pseudo_a_name}_${pseudo_cnt}"  synthetic_origin_rpy="${synthetic4_origin_r} ${synthetic4_origin_p} ${synthetic4_origin_ry}" synthetic_origin_xyz="${synthetic4_origin_x} ${synthetic4_origin_y} ${synthetic4_origin_z}" synthetic_parent="${pseudo_b_name}_${last_pseudo_cnt}" synthetic_child="${pseudo_a_name}_${pseudo_cnt}" />
+				<!-- Start building Pseudojoint 1 STATIC PART-->
+				<xacro:pseudo_static_link_mesh name="${pseudo_a_name}_${pseudo_cnt}" origin_xyz="${pseudo_a_origin_xyz}" origin_rpy="${pseudo_a_origin_rpy}"/>
 				<!-- PSEUDO2 CONFIGURATION -->
-				<xacro:pseudo_joint_name  pseudo_name="${pseudo_a_name}_3__${pseudo_b_name}_3"  pseudo_origin_rpy="${pseudo_origin_r+pseudo3_angle} ${pseudo_origin_p} ${pseudo_origin_y}" pseudo_origin_xyz="${pseudo_origin_xyz}" pseudo_parent="${pseudo_a_name}_3" pseudo_child="${pseudo_b_name}_3" />
-				<!-- Start building Pseudojoint 3 MOVING PART-->
-				<xacro:pseudo_moving_link_mesh name="${pseudo_b_name}_3" origin_xyz="${pseudo_b_origin_xyz}" origin_rpy="${pseudo_b_origin_rpy}"/>
-			</xacro:if>
-			<xacro:if value="${s5 == 21}">
-				<xacro:synthetic_joint_name  synthetic_name="${active_b_name}_1__${pseudo_a_name}_3"  synthetic_origin_rpy="${synthetic5_origin_r} ${synthetic5_origin_p} ${synthetic5_origin_ry}" synthetic_origin_xyz="${synthetic5_origin_x} ${synthetic5_origin_y} ${synthetic5_origin_z}" synthetic_parent="${active_b_name}_1" synthetic_child="${pseudo_a_name}_3" />
-				<!-- Start building Pseudojoint 3 STATIC PART-->
-				<xacro:pseudo_static_link_mesh name="${pseudo_a_name}_3" origin_xyz="${pseudo_a_origin_xyz}" origin_rpy="${pseudo_a_origin_rpy}"/>
+				<xacro:pseudo_joint_name  pseudo_name="${pseudo_a_name}_${pseudo_cnt}__${pseudo_b_name}_${pseudo_cnt}"  pseudo_origin_rpy="${pseudo_origin_r+pseudo2_angle} ${pseudo_origin_p} ${pseudo_origin_y}" pseudo_origin_xyz="${pseudo_origin_xyz}" pseudo_parent="${pseudo_a_name}_${pseudo_cnt}" pseudo_child="${pseudo_b_name}_${pseudo_cnt}" />
+				<!-- Start building Pseudojoint 1 MOVING PART-->
+				<xacro:pseudo_moving_link_mesh name="${pseudo_b_name}_${pseudo_cnt}" origin_xyz="${pseudo_b_origin_xyz}" origin_rpy="${pseudo_b_origin_rpy}"/>
+			</xacro:if>
+			<xacro:if value="${s6 == 31}">
+				<xacro:synthetic_joint_name  synthetic_name="${pseudo_b_name}_${last_pseudo_cnt}__${pseudo_a_name}_${pseudo_cnt}"  synthetic_origin_rpy="${synthetic2_origin_r} ${synthetic2_origin_p} ${synthetic2_origin_ry}" synthetic_origin_xyz="${synthetic2_origin_x} ${synthetic2_origin_y} ${synthetic2_origin_z}" synthetic_parent="${pseudo_b_name}_${last_pseudo_cnt}" synthetic_child="${pseudo_a_name}_${pseudo_cnt}" />
+				<!-- Start building Pseudojoint 2 STATIC PART-->
+				<xacro:pseudo_static_link_mesh name="${pseudo_a_name}_${pseudo_cnt}" origin_xyz="${pseudo_a_origin_xyz}" origin_rpy="${pseudo_a_origin_rpy}"/>
 				<!-- PSEUDO2 CONFIGURATION -->
-				<xacro:pseudo_joint_name  pseudo_name="${pseudo_a_name}_3__${pseudo_b_name}_3"  pseudo_origin_rpy="${pseudo_origin_r+pseudo3_angle} ${pseudo_origin_p} ${pseudo_origin_y}" pseudo_origin_xyz="${pseudo_origin_xyz}" pseudo_parent="${pseudo_a_name}_3" pseudo_child="${pseudo_b_name}_3" />
-				<!-- Start building Pseudojoint 3 MOVING PART-->
-				<xacro:pseudo_moving_link_mesh name="${pseudo_b_name}_3" origin_xyz="${pseudo_b_origin_xyz}" origin_rpy="${pseudo_b_origin_rpy}"/>
-			</xacro:if>
+				<xacro:pseudo_joint_name  pseudo_name="${pseudo_a_name}_${pseudo_cnt}__${pseudo_b_name}_${pseudo_cnt}"  pseudo_origin_rpy="${pseudo_origin_r+pseudo2_angle} ${pseudo_origin_p} ${pseudo_origin_y}" pseudo_origin_xyz="${pseudo_origin_xyz}" pseudo_parent="${pseudo_a_name}_${pseudo_cnt}" pseudo_child="${pseudo_b_name}_${pseudo_cnt}" />
+				<!-- Start building Pseudojoint 2 MOVING PART-->
+				<xacro:pseudo_moving_link_mesh name="${pseudo_b_name}_${pseudo_cnt}" origin_xyz="${pseudo_b_origin_xyz}" origin_rpy="${pseudo_b_origin_rpy}"/>
+			</xacro:if>
+		</xacro:unless>
+	</xacro:unless>
+	<xacro:if value="${s2 == 9 or s3==9}"> <!--  Second sub-case is previous meta link had 1 pseudo-->
+		<xacro:property name="last_pseudo_cnt" value="1" />
+		<xacro:property name="pseudo_cnt" value="2" />
+		<xacro:if value="${s5 == 31}">
+			<xacro:synthetic_joint_name  synthetic_name="${active_b_name}_${active_cnt}__${pseudo_a_name}_${pseudo_cnt}"  synthetic_origin_rpy="${synthetic3_origin_r} ${synthetic3_origin_p} ${synthetic3_origin_ry}" synthetic_origin_xyz="${synthetic3_origin_x} ${synthetic3_origin_y} ${synthetic3_origin_z}" synthetic_parent="${active_b_name}_${active_cnt}" synthetic_child="${pseudo_a_name}_${pseudo_cnt}" />
+			<!-- Start building Pseudojoint 3 STATIC PART-->
+			<xacro:pseudo_static_link_mesh name="${pseudo_a_name}_${pseudo_cnt}" origin_xyz="${pseudo_a_origin_xyz}" origin_rpy="${pseudo_a_origin_rpy}"/>
+			<!-- PSEUDO2 CONFIGURATION -->
+			<xacro:pseudo_joint_name  pseudo_name="${pseudo_a_name}_${pseudo_cnt}__${pseudo_b_name}_${pseudo_cnt}"  pseudo_origin_rpy="${pseudo_origin_r+pseudo3_angle} ${pseudo_origin_p} ${pseudo_origin_y}" pseudo_origin_xyz="${pseudo_origin_xyz}" pseudo_parent="${pseudo_a_name}_${pseudo_cnt}" pseudo_child="${pseudo_b_name}_${pseudo_cnt}" />
+			<!-- Start building Pseudojoint 3 MOVING PART-->
+			<xacro:pseudo_moving_link_mesh name="${pseudo_b_name}_${pseudo_cnt}" origin_xyz="${pseudo_b_origin_xyz}" origin_rpy="${pseudo_b_origin_rpy}"/>
+		</xacro:if>
+		<xacro:if value="${s5 == 21}">
+			<xacro:synthetic_joint_name  synthetic_name="${active_b_name}_${active_cnt}__${pseudo_a_name}_${pseudo_cnt}"  synthetic_origin_rpy="${synthetic5_origin_r} ${synthetic5_origin_p} ${synthetic5_origin_ry}" synthetic_origin_xyz="${synthetic5_origin_x} ${synthetic5_origin_y} ${synthetic5_origin_z}" synthetic_parent="${active_b_name}_${active_cnt}" synthetic_child="${pseudo_a_name}_${pseudo_cnt}" />
+			<!-- Start building Pseudojoint 3 STATIC PART-->
+			<xacro:pseudo_static_link_mesh name="${pseudo_a_name}_${pseudo_cnt}" origin_xyz="${pseudo_a_origin_xyz}" origin_rpy="${pseudo_a_origin_rpy}"/>
+			<!-- PSEUDO2 CONFIGURATION -->
+			<xacro:pseudo_joint_name  pseudo_name="${pseudo_a_name}_${pseudo_cnt}__${pseudo_b_name}_${pseudo_cnt}"  pseudo_origin_rpy="${pseudo_origin_r+pseudo3_angle} ${pseudo_origin_p} ${pseudo_origin_y}" pseudo_origin_xyz="${pseudo_origin_xyz}" pseudo_parent="${pseudo_a_name}_${pseudo_cnt}" pseudo_child="${pseudo_b_name}_${pseudo_cnt}" />
+			<!-- Start building Pseudojoint 3 MOVING PART-->
+			<xacro:pseudo_moving_link_mesh name="${pseudo_b_name}_${pseudo_cnt}" origin_xyz="${pseudo_b_origin_xyz}" origin_rpy="${pseudo_b_origin_rpy}"/>
+		</xacro:if>
+		<!-- Now evaluate next string of meta link!-->
+		<xacro:unless value="${s6 == 9}">
+			<xacro:property name="last_pseudo_cnt" value="2" />
+			<xacro:property name="pseudo_cnt" value="3" />
+			<xacro:if value="${s6 == 21}">
+				<xacro:synthetic_joint_name  synthetic_name="${pseudo_b_name}_${last_pseudo_cnt}__${pseudo_a_name}_${pseudo_cnt}"  synthetic_origin_rpy="${synthetic4_origin_r} ${synthetic4_origin_p} ${synthetic4_origin_ry}" synthetic_origin_xyz="${synthetic4_origin_x} ${synthetic4_origin_y} ${synthetic4_origin_z}" synthetic_parent="${pseudo_b_name}_${last_pseudo_cnt}" synthetic_child="${pseudo_a_name}_${pseudo_cnt}" />
+				<!-- Start building Pseudojoint 1 STATIC PART-->
+				<xacro:pseudo_static_link_mesh name="${pseudo_a_name}_${pseudo_cnt}" origin_xyz="${pseudo_a_origin_xyz}" origin_rpy="${pseudo_a_origin_rpy}"/>
+				<!-- PSEUDO2 CONFIGURATION -->
+				<xacro:pseudo_joint_name  pseudo_name="${pseudo_a_name}_${pseudo_cnt}__${pseudo_b_name}_${pseudo_cnt}"  pseudo_origin_rpy="${pseudo_origin_r+pseudo2_angle} ${pseudo_origin_p} ${pseudo_origin_y}" pseudo_origin_xyz="${pseudo_origin_xyz}" pseudo_parent="${pseudo_a_name}_${pseudo_cnt}" pseudo_child="${pseudo_b_name}_${pseudo_cnt}" />
+				<!-- Start building Pseudojoint 1 MOVING PART-->
+				<xacro:pseudo_moving_link_mesh name="${pseudo_b_name}_${pseudo_cnt}" origin_xyz="${pseudo_b_origin_xyz}" origin_rpy="${pseudo_b_origin_rpy}"/>
+			</xacro:if>
+			<xacro:if value="${s6 == 31}">
+				<xacro:synthetic_joint_name  synthetic_name="${pseudo_b_name}_${last_pseudo_cnt}__${pseudo_a_name}_${pseudo_cnt}"  synthetic_origin_rpy="${synthetic2_origin_r} ${synthetic2_origin_p} ${synthetic2_origin_ry}" synthetic_origin_xyz="${synthetic2_origin_x} ${synthetic2_origin_y} ${synthetic2_origin_z}" synthetic_parent="${pseudo_b_name}_${last_pseudo_cnt}" synthetic_child="${pseudo_a_name}_${pseudo_cnt}" />
+				<!-- Start building Pseudojoint 2 STATIC PART-->
+				<xacro:pseudo_static_link_mesh name="${pseudo_a_name}_${pseudo_cnt}" origin_xyz="${pseudo_a_origin_xyz}" origin_rpy="${pseudo_a_origin_rpy}"/>
+				<!-- PSEUDO2 CONFIGURATION -->
+				<xacro:pseudo_joint_name  pseudo_name="${pseudo_a_name}_${pseudo_cnt}__${pseudo_b_name}_${pseudo_cnt}"  pseudo_origin_rpy="${pseudo_origin_r+pseudo2_angle} ${pseudo_origin_p} ${pseudo_origin_y}" pseudo_origin_xyz="${pseudo_origin_xyz}" pseudo_parent="${pseudo_a_name}_${pseudo_cnt}" pseudo_child="${pseudo_b_name}_${pseudo_cnt}" />
+				<!-- Start building Pseudojoint 2 MOVING PART-->
+				<xacro:pseudo_moving_link_mesh name="${pseudo_b_name}_${pseudo_cnt}" origin_xyz="${pseudo_b_origin_xyz}" origin_rpy="${pseudo_b_origin_rpy}"/>
+			</xacro:if>
+		</xacro:unless>
+	</xacro:if>
 </xacro:unless>
+<xacro:if value="${s5 == 9}">  <!--  Second case is this meta link had no-pseudo in first string parameter => Builds next string-->
+	<xacro:unless value="${s2 == 9 and s3==9}"> <!--  First sub-case is previous meta link had 2 pseudos-->
+		<xacro:property name="last_pseudo_cnt" value="2" />
+		<xacro:property name="pseudo_cnt" value="3" />
+		<xacro:if value="${s6 == 31}">
+			<xacro:synthetic_joint_name  synthetic_name="${active_b_name}_${active_cnt}__${pseudo_a_name}_${pseudo_cnt}"  synthetic_origin_rpy="${synthetic3_origin_r} ${synthetic3_origin_p} ${synthetic3_origin_ry}" synthetic_origin_xyz="${synthetic3_origin_x} ${synthetic3_origin_y} ${synthetic3_origin_z}" synthetic_parent="${active_b_name}_${active_cnt}" synthetic_child="${pseudo_a_name}_${pseudo_cnt}" />
+			<!-- Start building Pseudojoint 3 STATIC PART-->
+			<xacro:pseudo_static_link_mesh name="${pseudo_a_name}_${pseudo_cnt}" origin_xyz="${pseudo_a_origin_xyz}" origin_rpy="${pseudo_a_origin_rpy}"/>
+			<!-- PSEUDO2 CONFIGURATION -->
+			<xacro:pseudo_joint_name  pseudo_name="${pseudo_a_name}_${pseudo_cnt}__${pseudo_b_name}_${pseudo_cnt}"  pseudo_origin_rpy="${pseudo_origin_r+pseudo3_angle} ${pseudo_origin_p} ${pseudo_origin_y}" pseudo_origin_xyz="${pseudo_origin_xyz}" pseudo_parent="${pseudo_a_name}_${pseudo_cnt}" pseudo_child="${pseudo_b_name}_${pseudo_cnt}" />
+			<!-- Start building Pseudojoint 3 MOVING PART-->
+			<xacro:pseudo_moving_link_mesh name="${pseudo_b_name}_${pseudo_cnt}" origin_xyz="${pseudo_b_origin_xyz}" origin_rpy="${pseudo_b_origin_rpy}"/>
+		</xacro:if>
+		<xacro:if value="${s6 == 21}">
+			<xacro:synthetic_joint_name  synthetic_name="${active_b_name}_${active_cnt}__${pseudo_a_name}_${pseudo_cnt}"  synthetic_origin_rpy="${synthetic5_origin_r} ${synthetic5_origin_p} ${synthetic5_origin_ry}" synthetic_origin_xyz="${synthetic5_origin_x} ${synthetic5_origin_y} ${synthetic5_origin_z}" synthetic_parent="${active_b_name}_${active_cnt}" synthetic_child="${pseudo_a_name}_${pseudo_cnt}" />
+			<!-- Start building Pseudojoint 3 STATIC PART-->
+			<xacro:pseudo_static_link_mesh name="${pseudo_a_name}_${pseudo_cnt}" origin_xyz="${pseudo_a_origin_xyz}" origin_rpy="${pseudo_a_origin_rpy}"/>
+			<!-- PSEUDO2 CONFIGURATION -->
+			<xacro:pseudo_joint_name  pseudo_name="${pseudo_a_name}_${pseudo_cnt}__${pseudo_b_name}_${pseudo_cnt}"  pseudo_origin_rpy="${pseudo_origin_r+pseudo3_angle} ${pseudo_origin_p} ${pseudo_origin_y}" pseudo_origin_xyz="${pseudo_origin_xyz}" pseudo_parent="${pseudo_a_name}_${pseudo_cnt}" pseudo_child="${pseudo_b_name}_${pseudo_cnt}" />
+			<!-- Start building Pseudojoint 3 MOVING PART-->
+			<xacro:pseudo_moving_link_mesh name="${pseudo_b_name}_${pseudo_cnt}" origin_xyz="${pseudo_b_origin_xyz}" origin_rpy="${pseudo_b_origin_rpy}"/>
+		</xacro:if>
+	</xacro:unless>
+	<xacro:if value="${s2 == 9 or s3==9}"> <!--  Second sub-case is previous meta link had 1 pseudo-->
+		<xacro:property name="last_pseudo_cnt" value="1" />
+		<xacro:property name="pseudo_cnt" value="2" />
+		<xacro:if value="${s6 == 31}">
+			<xacro:synthetic_joint_name  synthetic_name="${active_b_name}_${active_cnt}__${pseudo_a_name}_${pseudo_cnt}"  synthetic_origin_rpy="${synthetic3_origin_r} ${synthetic3_origin_p} ${synthetic3_origin_ry}" synthetic_origin_xyz="${synthetic3_origin_x} ${synthetic3_origin_y} ${synthetic3_origin_z}" synthetic_parent="${active_b_name}_${active_cnt}" synthetic_child="${pseudo_a_name}_${pseudo_cnt}" />
+			<!-- Start building Pseudojoint 3 STATIC PART-->
+			<xacro:pseudo_static_link_mesh name="${pseudo_a_name}_${pseudo_cnt}" origin_xyz="${pseudo_a_origin_xyz}" origin_rpy="${pseudo_a_origin_rpy}"/>
+			<!-- PSEUDO2 CONFIGURATION -->
+			<xacro:pseudo_joint_name  pseudo_name="${pseudo_a_name}_${pseudo_cnt}__${pseudo_b_name}_${pseudo_cnt}"  pseudo_origin_rpy="${pseudo_origin_r+pseudo3_angle} ${pseudo_origin_p} ${pseudo_origin_y}" pseudo_origin_xyz="${pseudo_origin_xyz}" pseudo_parent="${pseudo_a_name}_${pseudo_cnt}" pseudo_child="${pseudo_b_name}_${pseudo_cnt}" />
+			<!-- Start building Pseudojoint 3 MOVING PART-->
+			<xacro:pseudo_moving_link_mesh name="${pseudo_b_name}_${pseudo_cnt}" origin_xyz="${pseudo_b_origin_xyz}" origin_rpy="${pseudo_b_origin_rpy}"/>
+		</xacro:if>
+		<xacro:if value="${s6 == 21}">
+			<xacro:synthetic_joint_name  synthetic_name="${active_b_name}_${active_cnt}__${pseudo_a_name}_${pseudo_cnt}"  synthetic_origin_rpy="${synthetic5_origin_r} ${synthetic5_origin_p} ${synthetic5_origin_ry}" synthetic_origin_xyz="${synthetic5_origin_x} ${synthetic5_origin_y} ${synthetic5_origin_z}" synthetic_parent="${active_b_name}_${active_cnt}" synthetic_child="${pseudo_a_name}_${pseudo_cnt}" />
+			<!-- Start building Pseudojoint 3 STATIC PART-->
+			<xacro:pseudo_static_link_mesh name="${pseudo_a_name}_${pseudo_cnt}" origin_xyz="${pseudo_a_origin_xyz}" origin_rpy="${pseudo_a_origin_rpy}"/>
+			<!-- PSEUDO2 CONFIGURATION -->
+			<xacro:pseudo_joint_name  pseudo_name="${pseudo_a_name}_${pseudo_cnt}__${pseudo_b_name}_${pseudo_cnt}"  pseudo_origin_rpy="${pseudo_origin_r+pseudo3_angle} ${pseudo_origin_p} ${pseudo_origin_y}" pseudo_origin_xyz="${pseudo_origin_xyz}" pseudo_parent="${pseudo_a_name}_${pseudo_cnt}" pseudo_child="${pseudo_b_name}_${pseudo_cnt}" />
+			<!-- Start building Pseudojoint 3 MOVING PART-->
+			<xacro:pseudo_moving_link_mesh name="${pseudo_b_name}_${pseudo_cnt}" origin_xyz="${pseudo_b_origin_xyz}" origin_rpy="${pseudo_b_origin_rpy}"/>
+		</xacro:if>
+	</xacro:if>
+</xacro:if>
 </robot>

File: xacros/generated_urdf_from_xacros_here/conditioned_parameterized_SMM_assembly.urdf (robot description, URDF)
Before this commit: robot ovidius_smm, 8 links, 7 joints
Links:
- added link pseudo_a_2, mass 2.2036439; visual mesh filename=/home/nikos/PhD/projects/Parametric_Simulation_Model_SMM/Ps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 scale=0.001 0.001 0.001
- added link pseudo_a_4, mass 2.2036439; visual mesh filename=/home/nikos/PhD/projects/Parametric_Simulation_Model_SMM/Ps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 scale=0.001 0.001 0.001
- added link pseudo_b_2, mass 0.4450127; visual mesh filename=/home/nikos/PhD/projects/Parametric_Simulation_Model_SMM/Ps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 scale=0.001 0.001 0.001
- added link pseudo_b_4, mass 0.4450127; visual mesh filename=/home/nikos/PhD/projects/Parametric_Simulation_Model_SMM/Ps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 scale=0.001 0.001 0.001
Joints:
- removed joint pseudo_b_1__active_module_a_1
- added joint pseudo_a_2__pseudo_b_2: type fixed, parent pseudo_a_2, child pseudo_b_2, origin xyz=0 0.025 0.118 rpy=1.5708 0 0
- added joint pseudo_a_4__pseudo_b_4: type fixed, parent pseudo_a_4, child pseudo_b_4, origin xyz=0 0.025 0.118 rpy=1.5708 0 0
- added joint pseudo_b_1__pseudo_a_2: type fixed, parent pseudo_b_1, child pseudo_a_2, origin xyz=0 0.101 0 rpy=-1.5708 1.5708 0
- added joint pseudo_b_2__active_module_a_1: type fixed, parent pseudo_b_2, child active_module_a_1, origin xyz=0 0.1 0 rpy=0 1.5708 0
- added joint pseudo_b_3__pseudo_a_4: type fixed, parent pseudo_b_3, child pseudo_a_4, origin xyz=0 0.101 0 rpy=-1.5708 1.5708 0

Commit message: modified synthetic joint for dxl_frame2pseudo_back

File: xacros/conditioned_parameterized_SMM_assembly.xacro (robot description, xacro)
@@ -22,9 +22,9 @@
 <xacro:property name="synthetic3" value="${load_yaml(definitions_file)}"/>
 <xacro:property name="synthetic3_name" value="${synthetic3['synthetic3_name']}" />
-<xacro:property name="synthetic3_origin_x" value="${synthetic3['synthetic3_origin_x']}" />
+<!--xacro:property name="synthetic3_origin_x" value="${synthetic3['synthetic3_origin_x']}" / -->
 <xacro:property name="synthetic3_origin_y" value="${synthetic3['synthetic3_origin_y']}" />
 <!--xacro:property name="synthetic3_origin_z" value="${synthetic3['synthetic3_origin_z']}" / -->
 <xacro:property name="synthetic3_origin_r" value="${synthetic3['synthetic3_origin_r']}" />
-<xacro:property name="synthetic3_origin_p" value="${synthetic3['synthetic3_origin_p']}" />
+<!-- xacro:property name="synthetic3_origin_p" value="${synthetic3['synthetic3_origin_p']}" / -->
 <xacro:property name="synthetic3_origin_ry" value="${synthetic3['synthetic3_origin_ry']}" />
 <xacro:property name="synthetic4" value="${load_yaml(definitions_file)}"/>
@@ -100,6 +100,7 @@
 <xacro:property name="synthetic2_origin_x" value="${assembly_parameters['synthetic2_origin_x']}" />
 <xacro:property name="synthetic2_origin_p" value="${assembly_parameters['synthetic2_origin_p']}" />
+<xacro:property name="synthetic3_origin_x" value="${assembly_parameters['synthetic3_origin_x']}" />
 <xacro:property name="synthetic3_origin_z" value="${assembly_parameters['synthetic3_origin_z']}" />
-<!--xacro:property name="synthetic3_origin_ry" value="${assembly_parameters['synthetic3_origin_ry']}" /-->
+<xacro:property name="synthetic3_origin_p" value="${assembly_parameters['synthetic3_origin_p']}" />
 <xacro:property name="synthetic4_origin_x" value="${assembly_parameters['synthetic4_origin_x']}" />
 <xacro:property name="synthetic4_origin_p" value="${assembly_parameters['synthetic4_origin_p']}" />

File: xacros/generated_urdf_from_xacros_here/conditioned_parameterized_SMM_assembly.urdf (robot description, URDF)
Before this commit: robot ovidius_smm, 12 links, 11 joints
Joints:
- joint active_module_b_1__pseudo_a_3: origin xyz=0 0.0955 -0.05 rpy=0 0 0 -> xyz=-0.055 0.0955 -0.05 rpy=0 1.5708 0
- joint pseudo_b_1__pseudo_a_2: origin xyz=0 0.101 0 rpy=-1.5708 1.5708 0 -> xyz=-0.075 0.1444 0 rpy=0 1.5708 0
- joint pseudo_b_3__pseudo_a_4: origin xyz=0 0.101 0 rpy=-1.5708 1.5708 0 -> xyz=-0.075 0.1444 0 rpy=0 1.5708 0
