Commit message: added 3rd active joint in xacro

File: xacros/conditioned_parameterized_SMM_assembly.xacro (robot description, xacro)
@@ -340,3 +340,15 @@
 	</xacro:if>
 </xacro:if>
+<!-- ADD THIRD ROBOT JOINT->SECOND DYNAMIXEL JOINT -->
+<!-- This fixed tf assembles active module of link to preceding pseudo-->
+<xacro:if value="${s7 == 0}">
+	<xacro:property name="active_cnt" value="2" />
+	<xacro:assembly_active_module2pseudo  active_assembly_name="${pseudo_b_name}_${pseudo_cnt}__${active_a_name}_${active_cnt}"  active_assembly_origin_rpy="${active2pseudo_origin_rpy}" active_assembly_origin_xyz="${active2pseudo_origin_xyz}" active_assembly_parent="${pseudo_b_name}_${pseudo_cnt}" active_assembly_child="${active_a_name}_${active_cnt}" />
+	<!-- Adds Active Module STATIC PART-->
+	<xacro:active_static_link_mesh name="${active_a_name}_${active_cnt}" origin_xyz="${active_a_origin_xyz}" origin_rpy="${active_a_origin_rpy}"/>
+	<!-- Adds DXL Active joint -->
+	<xacro:dxlPROp_joint active_name="${active_a_name}_${active_cnt}__${active_b_name}_${active_cnt}"  active_origin_rpy="${active_origin_rpy}" active_origin_xyz="${active_origin_xyz}" active_parent="${active_a_name}_${active_cnt}" active_child="${active_b_name}_${active_cnt}"/>
+	<!-- Adds Active Module MOVING PART-->
+	<xacro:active_moving_link_mesh name="${active_b_name}_${active_cnt}" origin_xyz="${active_b_origin_xyz}" origin_rpy="${active_b_origin_rpy}"/>
+</xacro:if>
 </robot>

File: xacros/generated_urdf_from_xacros_here/conditioned_parameterized_SMM_assembly.urdf (robot description, URDF)
Before this commit: robot ovidius_smm, 12 links, 11 joints
Links:
- added link active_module_a_2, mass 0.892; visual mesh filename=/home/nikos/PhD/projects/Parametric_Simulation_Model_SMM/Ac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 scale=0.001 0.001 0.001
- added link active_module_b_2, mass 0.102; visual mesh filename=/home/nikos/PhD/projects/Parametric_Simulation_Model_SMM/Ac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 scale=0.001 0.001 0.001
Joints:
- added joint active_module_a_2__active_module_b_2: type revolute, parent active_module_a_2, child active_module_b_2, origin xyz=0 0.032 0 rpy=0 0 0, axis 0 0 1, limit lower=-2 upper=2 effort=55 velocity=4.0841
- added joint pseudo_b_4__active_module_a_2: type fixed, parent pseudo_b_4, child active_module_a_2, origin xyz=0 0.1 0 rpy=0 1.5708 0
- joint active_module_b_1__pseudo_a_3: origin xyz=-0.055 0.0955 -0.05 rpy=0 1.5708 0 -> xyz=0 0.0525 -0.015 rpy=-1.5708 0 0

Commit message: fixed bugs in pseudo angles at each assembly condition

File: xacros/conditioned_parameterized_SMM_assembly.xacro (robot description, xacro)
@@ -63,7 +63,8 @@
 <xacro:property name="pseudo_cnt" value="0" />
 <xacro:property name="last_pseudo_cnt" value="0" />
-<xacro:property name="pseudo1_angle" value="0"/>
-<xacro:property name="pseudo2_angle" value="0"/>
-<xacro:property name="pseudo3_angle" value="0"/>
+<xacro:property name="pseudo1_angle" value="1"/>
+<xacro:property name="pseudo2_angle" value="-1"/>
+<xacro:property name="pseudo3_angle" value="1"/>
+<xacro:property name="pseudo4_angle" value="-1"/>
 <!-- ACTIVE2PSEUDOS FIXED TFs -->
 <xacro:property name="active2pseudo" value="${load_yaml(definitions_file)}"/>
@@ -233,5 +234,5 @@
 				<xacro:pseudo_static_link_mesh name="${pseudo_a_name}_${pseudo_cnt}" origin_xyz="${pseudo_a_origin_xyz}" origin_rpy="${pseudo_a_origin_rpy}"/>
 				<!-- PSEUDO2 CONFIGURATION -->
-				<xacro:pseudo_joint_name  pseudo_name="${pseudo_a_name}_${pseudo_cnt}__${pseudo_b_name}_${pseudo_cnt}"  pseudo_origin_rpy="${pseudo_origin_r+pseudo2_angle} ${pseudo_origin_p} ${pseudo_origin_y}" pseudo_origin_xyz="${pseudo_origin_xyz}" pseudo_parent="${pseudo_a_name}_${pseudo_cnt}" pseudo_child="${pseudo_b_name}_${pseudo_cnt}" />
+				<xacro:pseudo_joint_name  pseudo_name="${pseudo_a_name}_${pseudo_cnt}__${pseudo_b_name}_${pseudo_cnt}"  pseudo_origin_rpy="${pseudo_origin_r+pseudo4_angle} ${pseudo_origin_p} ${pseudo_origin_y}" pseudo_origin_xyz="${pseudo_origin_xyz}" pseudo_parent="${pseudo_a_name}_${pseudo_cnt}" pseudo_child="${pseudo_b_name}_${pseudo_cnt}" />
 				<!-- Start building Pseudojoint 1 MOVING PART-->
 				<xacro:pseudo_moving_link_mesh name="${pseudo_b_name}_${pseudo_cnt}" origin_xyz="${pseudo_b_origin_xyz}" origin_rpy="${pseudo_b_origin_rpy}"/>
@@ -242,5 +243,5 @@
 				<xacro:pseudo_static_link_mesh name="${pseudo_a_name}_${pseudo_cnt}" origin_xyz="${pseudo_a_origin_xyz}" origin_rpy="${pseudo_a_origin_rpy}"/>
 				<!-- PSEUDO2 CONFIGURATION -->
-				<xacro:pseudo_joint_name  pseudo_name="${pseudo_a_name}_${pseudo_cnt}__${pseudo_b_name}_${pseudo_cnt}"  pseudo_origin_rpy="${pseudo_origin_r+pseudo2_angle} ${pseudo_origin_p} ${pseudo_origin_y}" pseudo_origin_xyz="${pseudo_origin_xyz}" pseudo_parent="${pseudo_a_name}_${pseudo_cnt}" pseudo_child="${pseudo_b_name}_${pseudo_cnt}" />
+				<xacro:pseudo_joint_name  pseudo_name="${pseudo_a_name}_${pseudo_cnt}__${pseudo_b_name}_${pseudo_cnt}"  pseudo_origin_rpy="${pseudo_origin_r+pseudo4_angle} ${pseudo_origin_p} ${pseudo_origin_y}" pseudo_origin_xyz="${pseudo_origin_xyz}" pseudo_parent="${pseudo_a_name}_${pseudo_cnt}" pseudo_child="${pseudo_b_name}_${pseudo_cnt}" />
 				<!-- Start building Pseudojoint 2 MOVING PART-->
 				<xacro:pseudo_moving_link_mesh name="${pseudo_b_name}_${pseudo_cnt}" origin_xyz="${pseudo_b_origin_xyz}" origin_rpy="${pseudo_b_origin_rpy}"/>
@@ -256,5 +257,5 @@
 			<xacro:pseudo_static_link_mesh name="${pseudo_a_name}_${pseudo_cnt}" origin_xyz="${pseudo_a_origin_xyz}" origin_rpy="${pseudo_a_origin_rpy}"/>
 			<!-- PSEUDO2 CONFIGURATION -->
-			<xacro:pseudo_joint_name  pseudo_name="${pseudo_a_name}_${pseudo_cnt}__${pseudo_b_name}_${pseudo_cnt}"  pseudo_origin_rpy="${pseudo_origin_r+pseudo3_angle} ${pseudo_origin_p} ${pseudo_origin_y}" pseudo_origin_xyz="${pseudo_origin_xyz}" pseudo_parent="${pseudo_a_name}_${pseudo_cnt}" pseudo_child="${pseudo_b_name}_${pseudo_cnt}" />
+			<xacro:pseudo_joint_name  pseudo_name="${pseudo_a_name}_${pseudo_cnt}__${pseudo_b_name}_${pseudo_cnt}"  pseudo_origin_rpy="${pseudo_origin_r+pseudo2_angle} ${pseudo_origin_p} ${pseudo_origin_y}" pseudo_origin_xyz="${pseudo_origin_xyz}" pseudo_parent="${pseudo_a_name}_${pseudo_cnt}" pseudo_child="${pseudo_b_name}_${pseudo_cnt}" />
 			<!-- Start building Pseudojoint 3 MOVING PART-->
 			<xacro:pseudo_moving_link_mesh name="${pseudo_b_name}_${pseudo_cnt}" origin_xyz="${pseudo_b_origin_xyz}" origin_rpy="${pseudo_b_origin_rpy}"/>
@@ -265,5 +266,5 @@
 			<xacro:pseudo_static_link_mesh name="${pseudo_a_name}_${pseudo_cnt}" origin_xyz="${pseudo_a_origin_xyz}" origin_rpy="${pseudo_a_origin_rpy}"/>
 			<!-- PSEUDO2 CONFIGURATION -->
-			<xacro:pseudo_joint_name  pseudo_name="${pseudo_a_name}_${pseudo_cnt}__${pseudo_b_name}_${pseudo_cnt}"  pseudo_origin_rpy="${pseudo_origin_r+pseudo3_angle} ${pseudo_origin_p} ${pseudo_origin_y}" pseudo_origin_xyz="${pseudo_origin_xyz}" pseudo_parent="${pseudo_a_name}_${pseudo_cnt}" pseudo_child="${pseudo_b_name}_${pseudo_cnt}" />
+			<xacro:pseudo_joint_name  pseudo_name="${pseudo_a_name}_${pseudo_cnt}__${pseudo_b_name}_${pseudo_cnt}"  pseudo_origin_rpy="${pseudo_origin_r+pseudo2_angle} ${pseudo_origin_p} ${pseudo_origin_y}" pseudo_origin_xyz="${pseudo_origin_xyz}" pseudo_parent="${pseudo_a_name}_${pseudo_cnt}" pseudo_child="${pseudo_b_name}_${pseudo_cnt}" />
 			<!-- Start building Pseudojoint 3 MOVING PART-->
 			<xacro:pseudo_moving_link_mesh name="${pseudo_b_name}_${pseudo_cnt}" origin_xyz="${pseudo_b_origin_xyz}" origin_rpy="${pseudo_b_origin_rpy}"/>
@@ -278,5 +279,5 @@
 				<xacro:pseudo_static_link_mesh name="${pseudo_a_name}_${pseudo_cnt}" origin_xyz="${pseudo_a_origin_xyz}" origin_rpy="${pseudo_a_origin_rpy}"/>
 				<!-- PSEUDO2 CONFIGURATION -->
-				<xacro:pseudo_joint_name  pseudo_name="${pseudo_a_name}_${pseudo_cnt}__${pseudo_b_name}_${pseudo_cnt}"  pseudo_origin_rpy="${pseudo_origin_r+pseudo2_angle} ${pseudo_origin_p} ${pseudo_origin_y}" pseudo_origin_xyz="${pseudo_origin_xyz}" pseudo_parent="${pseudo_a_name}_${pseudo_cnt}" pseudo_child="${pseudo_b_name}_${pseudo_cnt}" />
+				<xacro:pseudo_joint_name  pseudo_name="${pseudo_a_name}_${pseudo_cnt}__${pseudo_b_name}_${pseudo_cnt}"  pseudo_origin_rpy="${pseudo_origin_r+pseudo3_angle} ${pseudo_origin_p} ${pseudo_origin_y}" pseudo_origin_xyz="${pseudo_origin_xyz}" pseudo_parent="${pseudo_a_name}_${pseudo_cnt}" pseudo_child="${pseudo_b_name}_${pseudo_cnt}" />
 				<!-- Start building Pseudojoint 1 MOVING PART-->
 				<xacro:pseudo_moving_link_mesh name="${pseudo_b_name}_${pseudo_cnt}" origin_xyz="${pseudo_b_origin_xyz}" origin_rpy="${pseudo_b_origin_rpy}"/>
@@ -287,5 +288,5 @@
 				<xacro:pseudo_static_link_mesh name="${pseudo_a_name}_${pseudo_cnt}" origin_xyz="${pseudo_a_origin_xyz}" origin_rpy="${pseudo_a_origin_rpy}"/>
 				<!-- PSEUDO2 CONFIGURATION -->
-				<xacro:pseudo_joint_name  pseudo_name="${pseudo_a_name}_${pseudo_cnt}__${pseudo_b_name}_${pseudo_cnt}"  pseudo_origin_rpy="${pseudo_origin_r+pseudo2_angle} ${pseudo_origin_p} ${pseudo_origin_y}" pseudo_origin_xyz="${pseudo_origin_xyz}" pseudo_parent="${pseudo_a_name}_${pseudo_cnt}" pseudo_child="${pseudo_b_name}_${pseudo_cnt}" />
+				<xacro:pseudo_joint_name  pseudo_name="${pseudo_a_name}_${pseudo_cnt}__${pseudo_b_name}_${pseudo_cnt}"  pseudo_origin_rpy="${pseudo_origin_r+pseudo3_angle} ${pseudo_origin_p} ${pseudo_origin_y}" pseudo_origin_xyz="${pseudo_origin_xyz}" pseudo_parent="${pseudo_a_name}_${pseudo_cnt}" pseudo_child="${pseudo_b_name}_${pseudo_cnt}" />
 				<!-- Start building Pseudojoint 2 MOVING PART-->
 				<xacro:pseudo_moving_link_mesh name="${pseudo_b_name}_${pseudo_cnt}" origin_xyz="${pseudo_b_origin_xyz}" origin_rpy="${pseudo_b_origin_rpy}"/>
@@ -325,5 +326,5 @@
 			<xacro:pseudo_static_link_mesh name="${pseudo_a_name}_${pseudo_cnt}" origin_xyz="${pseudo_a_origin_xyz}" origin_rpy="${pseudo_a_origin_rpy}"/>
 			<!-- PSEUDO2 CONFIGURATION -->
-			<xacro:pseudo_joint_name  pseudo_name="${pseudo_a_name}_${pseudo_cnt}__${pseudo_b_name}_${pseudo_cnt}"  pseudo_origin_rpy="${pseudo_origin_r+pseudo3_angle} ${pseudo_origin_p} ${pseudo_origin_y}" pseudo_origin_xyz="${pseudo_origin_xyz}" pseudo_parent="${pseudo_a_name}_${pseudo_cnt}" pseudo_child="${pseudo_b_name}_${pseudo_cnt}" />
+			<xacro:pseudo_joint_name  pseudo_name="${pseudo_a_name}_${pseudo_cnt}__${pseudo_b_name}_${pseudo_cnt}"  pseudo_origin_rpy="${pseudo_origin_r+pseudo2_angle} ${pseudo_origin_p} ${pseudo_origin_y}" pseudo_origin_xyz="${pseudo_origin_xyz}" pseudo_parent="${pseudo_a_name}_${pseudo_cnt}" pseudo_child="${pseudo_b_name}_${pseudo_cnt}" />
 			<!-- Start building Pseudojoint 3 MOVING PART-->
 			<xacro:pseudo_moving_link_mesh name="${pseudo_b_name}_${pseudo_cnt}" origin_xyz="${pseudo_b_origin_xyz}" origin_rpy="${pseudo_b_origin_rpy}"/>
@@ -334,5 +335,5 @@
 			<xacro:pseudo_static_link_mesh name="${pseudo_a_name}_${pseudo_cnt}" origin_xyz="${pseudo_a_origin_xyz}" origin_rpy="${pseudo_a_origin_rpy}"/>
 			<!-- PSEUDO2 CONFIGURATION -->
-			<xacro:pseudo_joint_name  pseudo_name="${pseudo_a_name}_${pseudo_cnt}__${pseudo_b_name}_${pseudo_cnt}"  pseudo_origin_rpy="${pseudo_origin_r+pseudo3_angle} ${pseudo_origin_p} ${pseudo_origin_y}" pseudo_origin_xyz="${pseudo_origin_xyz}" pseudo_parent="${pseudo_a_name}_${pseudo_cnt}" pseudo_child="${pseudo_b_name}_${pseudo_cnt}" />
+			<xacro:pseudo_joint_name  pseudo_name="${pseudo_a_name}_${pseudo_cnt}__${pseudo_b_name}_${pseudo_cnt}"  pseudo_origin_rpy="${pseudo_origin_r+pseudo2_angle} ${pseudo_origin_p} ${pseudo_origin_y}" pseudo_origin_xyz="${pseudo_origin_xyz}" pseudo_parent="${pseudo_a_name}_${pseudo_cnt}" pseudo_child="${pseudo_b_name}_${pseudo_cnt}" />
 			<!-- Start building Pseudojoint 3 MOVING PART-->
 			<xacro:pseudo_moving_link_mesh name="${pseudo_b_name}_${pseudo_cnt}" origin_xyz="${pseudo_b_origin_xyz}" origin_rpy="${pseudo_b_origin_rpy}"/>

File: xacros/generated_urdf_from_xacros_here/conditioned_parameterized_SMM_assembly.urdf (robot description, URDF)
Before this commit: robot ovidius_smm, 14 links, 13 joints
Joints:
- joint pseudo_a_1__pseudo_b_1: origin xyz=0 0.025 0.118 rpy=1.5708 0 0 -> xyz=0 0.025 0.118 rpy=2.5708 0 0
- joint pseudo_a_2__pseudo_b_2: origin xyz=0 0.025 0.118 rpy=1.5708 0 0 -> xyz=0 0.025 0.118 rpy=0.5708 0 0
- joint pseudo_a_3__pseudo_b_3: origin xyz=0 0.025 0.118 rpy=1.5708 0 0 -> xyz=0 0.025 0.118 rpy=2.5708 0 0
- joint pseudo_a_4__pseudo_b_4: origin xyz=0 0.025 0.118 rpy=1.5708 0 0 -> xyz=0 0.025 0.118 rpy=0.5708 0 0

Commit message: minor changes for testing  inertia values

File: xacros/conditioned_parameterized_SMM_assembly.xacro (robot description, xacro)
@@ -63,8 +63,8 @@
 <xacro:property name="pseudo_cnt" value="0" />
 <xacro:property name="last_pseudo_cnt" value="0" />
-<xacro:property name="pseudo1_angle" value="1"/>
-<xacro:property name="pseudo2_angle" value="-1"/>
-<xacro:property name="pseudo3_angle" value="1"/>
-<xacro:property name="pseudo4_angle" value="-1"/>
+<xacro:property name="pseudo1_angle" value="0"/>
+<xacro:property name="pseudo2_angle" value="0"/>
+<xacro:property name="pseudo3_angle" value="0"/>
+<xacro:property name="pseudo4_angle" value="0"/>
 <!-- ACTIVE2PSEUDOS FIXED TFs -->
 <xacro:property name="active2pseudo" value="${load_yaml(definitions_file)}"/>

File: xacros/generated_urdf_from_xacros_here/inertia_test_robot.urdf (robot description, URDF)
Before this commit: robot ovidius_smm, 12 links, 11 joints
Joints:
- joint pseudo_a_1__pseudo_b_1: origin xyz=0 0.025 0.118 rpy=2.5708 0 0 -> xyz=0 0.025 0.118 rpy=1.5708 0 0
- joint pseudo_a_2__pseudo_b_2: origin xyz=0 0.025 0.118 rpy=0.5708 0 0 -> xyz=0 0.025 0.118 rpy=1.5708 0 0
- joint pseudo_a_3__pseudo_b_3: origin xyz=0 0.025 0.118 rpy=2.5708 0 0 -> xyz=0 0.025 0.118 rpy=1.5708 0 0

File: xacros/generated_urdf_from_xacros_here/pseudo_module.urdf (robot description, URDF)
Before this commit: robot ovidius_v1, 4 links, 3 joints
Links:
- removed link base_link
Joints:
- removed joint base_link__PseudoConnector1a
- removed joint world__base_link
- added joint world__PseudoConnector1a: type revolute, parent world, child PseudoConnector1a, origin xyz=0 0 0 rpy=0 0 0, axis 0 0 1, limit lower=-2 upper=2 effort=55 velocity=4.0841

File: xacros/ovidius_links_joints_names.xacro (robot description, xacro)
@@ -11,5 +11,5 @@
     <link name="${name}">
       <inertial>
-        <origin rpy="0 0 0" xyz="0 0 0"/>
+        <origin rpy="0 0 0" xyz="0 0 0.09"/>
         <mass value ="${pseudo_mass_static}" />
         <inertia ixx="3.5655174315e-07" ixy="3.0094534019e-15" ixz="-3.0659548585e-16" iyy="8.1971725028e-7" iyz="1.0236492333e-16" izz="5.0684999189e-07"/>
@@ -30,5 +30,5 @@
     <link name="${name}">
       <inertial>
-        <origin rpy="0 0 0" xyz="0 0 0"/>
+        <origin rpy="0 0 0" xyz="0 0 0.04"/>
         <mass value ="${pseudo_mass_moving}" />
         <inertia ixx="1.345843e-07" ixy="1.399547e-14" ixz="-2.461662e-15" iyy="1.577317e-7" iyz="2.024057e-13" izz="1.101806e-7"/>

File: xacros/pseudo_module.xacro (robot description, xacro)
@@ -16,4 +16,5 @@
 <xacro:property name="fPz011" value="${0+Pz011}"/>
 <link name="world"/>
+<!--
 <joint name="world__base_link" type="fixed">
 <origin rpy="0 0 0" xyz="0 0 0"/>
@@ -37,7 +38,9 @@
     </visual>
 </link>
-  <joint name="base_link__PseudoConnector1a" type="revolute">
-    <origin rpy="${Rx011} ${Ry011} ${Rz011}" xyz="${fPx011} ${Py011} ${fPz011}"/>
-    <parent link="base_link"/>
+-->
+  <joint name="world__PseudoConnector1a" type="revolute">
+    <!--<origin rpy="${Rx011} ${Ry011} ${Rz011}" xyz="${fPx011} ${Py011} ${fPz011}"/>-->
+    <origin rpy="0 0 0" xyz="0 0 0"/>
+    <parent link="world"/>
     <child link="PseudoConnector1a"/>
     <!-- axis,limit,dynamics are only added here to be able to compute COM in matlab-->
@@ -48,5 +51,5 @@
 <link name="PseudoConnector1a">
       <inertial>
-        <origin rpy="0 0 0" xyz="0 0 0"/>
+        <origin rpy="0 0 0" xyz="0 0 0.09"/>
         <mass value ="${pseudo_mass_static}" />
         <inertia ixx="3.5655174315e-07" ixy="3.0094534019e-15" ixz="-3.0659548585e-16" iyy="8.1971725028e-7" iyz="1.0236492333e-16" izz="5.0684999189e-07"/>
@@ -71,5 +74,5 @@
 <link name="PseudoConnector1b">
     <inertial>
-      <origin rpy="0 0 0" xyz="0 0 0"/>
+      <origin rpy="0 0 0" xyz="0 0 0.04"/>
       <mass value ="${pseudo_mass_moving}" />
       <inertia ixx="1.345843e-07" ixy="1.399547e-14" ixz="-2.461662e-15" iyy="1.577317e-7" iyz="2.024057e-13" izz="1.101806e-7"/>

Commit message: started a 2dof project to help symbolics for matlab model

File: xacros/conditioned_parameterized_SMM_assembly.xacro (robot description, xacro)
@@ -63,8 +63,8 @@
 <xacro:property name="pseudo_cnt" value="0" />
 <xacro:property name="last_pseudo_cnt" value="0" />
-<xacro:property name="pseudo1_angle" value="0"/>
-<xacro:property name="pseudo2_angle" value="0"/>
-<xacro:property name="pseudo3_angle" value="0"/>
-<xacro:property name="pseudo4_angle" value="0"/>
+<xacro:property name="pseudo1_angle" value="1"/>
+<xacro:property name="pseudo2_angle" value="-1"/>
+<xacro:property name="pseudo3_angle" value="1"/>
+<xacro:property name="pseudo4_angle" value="-1"/>
 <!-- ACTIVE2PSEUDOS FIXED TFs -->
 <xacro:property name="active2pseudo" value="${load_yaml(definitions_file)}"/>
@@ -123,5 +123,5 @@
 <link name="base_link">
     <inertial>
-      <origin rpy="0 0 0" xyz="0.00205 0.00373 0.020774"/>
+      <origin rpy="0 0 0" xyz="0.00205 0.00373 0.015774"/>
       <mass value ="0.500" />
       <inertia ixx="5.063e-004" ixy="2.773e-005" ixz="7.042e-007" iyy="5.387e-004" iyz="1.237e-006" izz="7.207e-004"/>
@@ -352,4 +352,12 @@
 	<!-- Adds Active Module MOVING PART-->
 	<xacro:active_moving_link_mesh name="${active_b_name}_${active_cnt}" origin_xyz="${active_b_origin_xyz}" origin_rpy="${active_b_origin_rpy}"/>
+	<!-- Add TCP as TOOL frame-->
+	<!-- Add TCP -->
+	<joint name="${active_b_name}_${active_cnt}__TOOL" type="fixed">
+	    <origin rpy="0 0 0" xyz="0 0.05 0"/>
+	    <parent link="${active_b_name}_${active_cnt}"/>
+	    <child link="TOOL"/>
+	</joint>
+	<link name="TOOL"/>
 </xacro:if>
 </robot>

File: xacros/generated_urdf_from_xacros_here/conditioned_parameterized_SMM_assembly.urdf (robot description, URDF)
Before this commit: robot ovidius_smm, 12 links, 11 joints
Links:
- added link TOOL
- added link pseudo_a_4, mass 2.2036439; visual mesh filename=/home/nikos/PhD/projects/Parametric_Simulation_Model_SMM/Ps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 scale=0.001 0.001 0.001
- added link pseudo_b_4, mass 0.4450127; visual mesh filename=/home/nikos/PhD/projects/Parametric_Simulation_Model_SMM/Ps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 scale=0.001 0.001 0.001
Joints:
- removed joint active_module_b_1__pseudo_a_2
- removed joint pseudo_b_1__active_module_a_1
- removed joint pseudo_b_2__pseudo_a_3
- removed joint pseudo_b_3__active_module_a_2
- added joint active_module_b_1__pseudo_a_3: type fixed, parent active_module_b_1, child pseudo_a_3, origin xyz=0 0.0525 0 rpy=-1.5708 0 0
- added joint active_module_b_2__TOOL: type fixed, parent active_module_b_2, child TOOL, origin xyz=0 0.05 0 rpy=0 0 0
- added joint pseudo_a_4__pseudo_b_4: type fixed, parent pseudo_a_4, child pseudo_b_4, origin xyz=0 0.025 0.118 rpy=0.5708 0 0
- added joint pseudo_b_1__pseudo_a_2: type fixed, parent pseudo_b_1, child pseudo_a_2, origin xyz=-0.025 0.1444 -0.05 rpy=0 0 0
- added joint pseudo_b_2__active_module_a_1: type fixed, parent pseudo_b_2, child active_module_a_1, origin xyz=0 0.1 0 rpy=0 1.5708 0
- added joint pseudo_b_3__pseudo_a_4: type fixed, parent pseudo_b_3, child pseudo_a_4, origin xyz=-0.025 0.1444 -0.05 rpy=0 0 0
- added joint pseudo_b_4__active_module_a_2: type fixed, parent pseudo_b_4, child active_module_a_2, origin xyz=0 0.1 0 rpy=0 1.5708 0
