Commit message: solved issue on active2pseudo tf for active twist generation, added parametric modeling for active2pseudo assembly

File: xacros/conditioned_parameterized_SMM_assembly.xacro (robot description, xacro)
@@ -16,5 +16,5 @@
 <!-- xacro:property name="synthetic2_origin_x" value="${synthetic2['synthetic2_origin_x']}" / -->
 <xacro:property name="synthetic2_origin_y" value="${synthetic2['synthetic2_origin_y']}" />
-<xacro:property name="synthetic2_origin_z" value="${synthetic2['synthetic2_origin_z']}" />
+<!--xacro:property name="synthetic2_origin_z" value="${synthetic2['synthetic2_origin_z']}" / -->
 <xacro:property name="synthetic2_origin_r" value="${synthetic2['synthetic2_origin_r']}" />
 <!-- xacro:property name="synthetic2_origin_p" value="${synthetic2['synthetic2_origin_p']}" / -->
@@ -32,5 +32,5 @@
 <!-- xacro:property name="synthetic4_origin_x" value="${synthetic4['synthetic4_origin_x']}" / -->
 <xacro:property name="synthetic4_origin_y" value="${synthetic4['synthetic4_origin_y']}" />
-<xacro:property name="synthetic4_origin_z" value="${synthetic4['synthetic4_origin_z']}" />
+<!--xacro:property name="synthetic4_origin_z" value="${synthetic4['synthetic4_origin_z']}" / -->
 <xacro:property name="synthetic4_origin_r" value="${synthetic4['synthetic4_origin_r']}" />
 <!-- xacro:property name="synthetic4_origin_p" value="${synthetic4['synthetic4_origin_p']}" /-->
@@ -38,5 +38,5 @@
 <xacro:property name="synthetic5" value="${load_yaml(definitions_file)}"/>
 <xacro:property name="synthetic5_name" value="${synthetic5['synthetic5_name']}" />
-<xacro:property name="synthetic5_origin_x" value="${synthetic5['synthetic5_origin_x']}" />
+<!--xacro:property name="synthetic5_origin_x" value="${synthetic5['synthetic5_origin_x']}" /-->
 <xacro:property name="synthetic5_origin_y" value="${synthetic5['synthetic5_origin_y']}" />
 <!--xacro:property name="synthetic5_origin_z" value="${synthetic5['synthetic5_origin_z']}" /-->
@@ -63,13 +63,16 @@
 <xacro:property name="pseudo_cnt" value="0" />
 <xacro:property name="last_pseudo_cnt" value="0" />
-<xacro:property name="pseudo1_angle" value="1"/>
-<xacro:property name="pseudo2_angle" value="-1"/>
-<xacro:property name="pseudo3_angle" value="1"/>
-<xacro:property name="pseudo4_angle" value="-1"/>
+<xacro:property name="pseudo1_angle" value="0"/>
+<xacro:property name="pseudo2_angle" value="0"/>
+<xacro:property name="pseudo3_angle" value="0"/>
+<xacro:property name="pseudo4_angle" value="0"/>
 <!-- ACTIVE2PSEUDOS FIXED TFs -->
 <xacro:property name="active2pseudo" value="${load_yaml(definitions_file)}"/>
 <xacro:property name="active2pseudo_name" value="${active2pseudo['active2pseudo_name']}" />
 <xacro:property name="active2pseudo_origin_xyz" value="${active2pseudo['active2pseudo_origin_xyz']}" />
-<xacro:property name="active2pseudo_origin_rpy" value="${active2pseudo['active2pseudo_origin_rpy']}" />
+<!--xacro:property name="active2pseudo_origin_rpy" value="${active2pseudo['active2pseudo_origin_rpy']}" /-->
+<xacro:property name="active2pseudo_origin_r" value="${active2pseudo['active2pseudo_origin_r']}" />
+<!--xacro:property name="active2pseudo_origin_p" value="${active2pseudo['active2pseudo__origin__p']}" /-->
+<xacro:property name="active2pseudo_origin_ry" value="${active2pseudo['active2pseudo_origin_ry']}" />
 <!-- ACTIVE MODULE PARTS -->
 <xacro:property name="active_a" value="${load_yaml(definitions_file)}"/>
@@ -100,4 +103,5 @@
 <xacro:property name="assembly_parameters" value="${load_yaml(ovidius_assembly_parameters_file)}"/>
 <xacro:property name="synthetic2_origin_x" value="${assembly_parameters['synthetic2_origin_x']}" />
+<xacro:property name="synthetic2_origin_z" value="${assembly_parameters['synthetic2_origin_z']}" />
 <xacro:property name="synthetic2_origin_p" value="${assembly_parameters['synthetic2_origin_p']}" />
 <xacro:property name="synthetic3_origin_x" value="${assembly_parameters['synthetic3_origin_x']}" />
@@ -105,7 +109,10 @@
 <xacro:property name="synthetic3_origin_p" value="${assembly_parameters['synthetic3_origin_p']}" />
 <xacro:property name="synthetic4_origin_x" value="${assembly_parameters['synthetic4_origin_x']}" />
+<xacro:property name="synthetic4_origin_z" value="${assembly_parameters['synthetic4_origin_z']}" />
 <xacro:property name="synthetic4_origin_p" value="${assembly_parameters['synthetic4_origin_p']}" />
+<xacro:property name="synthetic5_origin_x" value="${assembly_parameters['synthetic5_origin_x']}" />
 <xacro:property name="synthetic5_origin_z" value="${assembly_parameters['synthetic5_origin_z']}" />
 <xacro:property name="synthetic5_origin_p" value="${assembly_parameters['synthetic5_origin_p']}" />
+<xacro:property name="active2pseudo_origin_p" value="${assembly_parameters['active2pseudo_origin_p']}" />
 <!-- III.1	ROBOT to be generated to URDF model-->
 <!-- ROBOT DESCRIPTION-->
@@ -194,5 +201,5 @@
 <xacro:if value="${s4 == 0}">
 	<xacro:property name="active_cnt" value="1" />
-	<xacro:assembly_active_module2pseudo  active_assembly_name="${pseudo_b_name}_${pseudo_cnt}__${active_a_name}_${active_cnt}"  active_assembly_origin_rpy="${active2pseudo_origin_rpy}" active_assembly_origin_xyz="${active2pseudo_origin_xyz}" active_assembly_parent="${pseudo_b_name}_${pseudo_cnt}" active_assembly_child="${active_a_name}_${active_cnt}" />
+	<xacro:assembly_active_module2pseudo  active_assembly_name="${pseudo_b_name}_${pseudo_cnt}__${active_a_name}_${active_cnt}"  active_assembly_origin_rpy="${active2pseudo_origin_r} ${active2pseudo_origin_p} ${active2pseudo_origin_ry}" active_assembly_origin_xyz="${active2pseudo_origin_xyz}" active_assembly_parent="${pseudo_b_name}_${pseudo_cnt}" active_assembly_child="${active_a_name}_${active_cnt}" />
 	<!-- Adds Active Module STATIC PART-->
 	<xacro:active_static_link_mesh name="${active_a_name}_${active_cnt}" origin_xyz="${active_a_origin_xyz}" origin_rpy="${active_a_origin_rpy}"/>
@@ -345,5 +352,5 @@
 <xacro:if value="${s7 == 0}">
 	<xacro:property name="active_cnt" value="2" />
-	<xacro:assembly_active_module2pseudo  active_assembly_name="${pseudo_b_name}_${pseudo_cnt}__${active_a_name}_${active_cnt}"  active_assembly_origin_rpy="${active2pseudo_origin_rpy}" active_assembly_origin_xyz="${active2pseudo_origin_xyz}" active_assembly_parent="${pseudo_b_name}_${pseudo_cnt}" active_assembly_child="${active_a_name}_${active_cnt}" />
+	<xacro:assembly_active_module2pseudo  active_assembly_name="${pseudo_b_name}_${pseudo_cnt}__${active_a_name}_${active_cnt}"  active_assembly_origin_rpy="${active2pseudo_origin_r} ${active2pseudo_origin_p} ${active2pseudo_origin_ry}" active_assembly_origin_xyz="${active2pseudo_origin_xyz}" active_assembly_parent="${pseudo_b_name}_${pseudo_cnt}" active_assembly_child="${active_a_name}_${active_cnt}" />
 	<!-- Adds Active Module STATIC PART-->
 	<xacro:active_static_link_mesh name="${active_a_name}_${active_cnt}" origin_xyz="${active_a_origin_xyz}" origin_rpy="${active_a_origin_rpy}"/>

File: xacros/generated_urdf_from_xacros_here/conditioned_parameterized_SMM_assembly.urdf (robot description, URDF)
Before this commit: robot ovidius_smm, 15 links, 14 joints
Joints:
- joint active_module_a_1__active_module_b_1: axis 0 0 1 -> 1 0 0; origin xyz=0 0.032 0 rpy=0 0 0 -> xyz=0 0.032 0 rpy=0 1.5708 0
- joint active_module_a_2__active_module_b_2: axis 0 0 1 -> 1 0 0; origin xyz=0 0.032 0 rpy=0 0 0 -> xyz=0 0.032 0 rpy=0 1.5708 0
- joint active_module_b_1__pseudo_a_3: origin xyz=0 0.0525 0 rpy=-1.5708 0 0 -> xyz=0.01 0.0525 0 rpy=-1.5708 0 0
- joint pseudo_a_1__pseudo_b_1: origin xyz=0 0.025 0.118 rpy=2.5708 0 0 -> xyz=0 0.025 0.118 rpy=1.5708 0 0
- joint pseudo_a_2__pseudo_b_2: origin xyz=0 0.025 0.118 rpy=0.5708 0 0 -> xyz=0 0.025 0.118 rpy=1.5708 0 0
- joint pseudo_a_3__pseudo_b_3: origin xyz=0 0.025 0.118 rpy=2.5708 0 0 -> xyz=0 0.025 0.118 rpy=1.5708 0 0
- joint pseudo_a_4__pseudo_b_4: origin xyz=0 0.025 0.118 rpy=0.5708 0 0 -> xyz=0 0.025 0.118 rpy=1.5708 0 0
- joint pseudo_b_1__pseudo_a_2: origin xyz=-0.025 0.1444 -0.05 rpy=0 0 0 -> xyz=-0.025 0.1444 0.01 rpy=0 0 0
- joint pseudo_b_2__active_module_a_1: origin xyz=0 0.1 0 rpy=0 1.5708 0 -> xyz=0 0.1 0 rpy=0 0 0
- joint pseudo_b_3__pseudo_a_4: origin xyz=-0.025 0.1444 -0.05 rpy=0 0 0 -> xyz=-0.025 0.1444 0.01 rpy=0 0 0
- joint pseudo_b_4__active_module_a_2: origin xyz=0 0.1 0 rpy=0 1.5708 0 -> xyz=0 0.1 0 rpy=0 0 0

File: xacros/ovidius_links_joints_names.xacro (robot description, xacro)
@@ -113,5 +113,5 @@
       <parent link="${active_parent}" />
       <child link="${active_child}" />
-      <axis xyz="0 0 1"/>
+      <axis xyz="1 0 0"/>
       <limit effort="55" lower="-2" upper="2" velocity="4.0841"/>
       <dynamics damping="0.5"/>
