Commit message: Working on 6dof assembly. Building the metalink_for_6dof_assembly

File: xacros/cases_overview_6dof_for_ga.xacro (robot description, xacro)
@@ -1,4 +1,8 @@
 <!-- CASES FOR METAMORPHIC LINK FOR DOF HIGHER THAN 3-->
-<xacro:unless value="${sj == 9}"> <!--  Case A is this meta link had pseudo in first string parameter-->
+<!-- This will be modified to a big boy xacro and added to the 6dof code -->
+<xacro:unless value="${sj == 9}"> <!--  Case A is this meta link had pseudo in first string parameter => ONLY CASE BECAUSE IN GA THE FIRST PSEUDO MUST ALWAYS EXIST!-->
+	// Give naming
+	// metalink_i
+	// metalink_i_pseudo1
 	<xacro:if value="${s_j == 31}"> <!-- Case A.1.a -->
 	</xacro:if>
@@ -6,4 +10,5 @@
 	</xacro:if>
 	<xacro:unless value="${s_j+1 == 9}"> <!-- Case A.1.c : and a 2nd pseudo exists-->
+		// metalink_i_pseudo2
 		<xacro:if value="${s_j+1 == 31}"> <!-- Case A.1.c.1 -->
 		</xacro:if>
@@ -11,3 +16,6 @@
 		</xacro:if>
 	</xacro:unless>
+	<xacro:if value="${s_j+1 == 9}"> <!-- Case A.1.d : if a 2nd pseudo doesn't exist-->
+	// Add nothing here
+	</xacro:if>
 </xacro:unless>	<!--  Case A - end-->

File: xacros/conditioned_parameterized_SMM_assembly_6dof_for_ga.xacro (robot description, xacro)
@@ -433,4 +433,8 @@
 <!-- #############################################################################################################################################-->
 <!-- STARTED 3RD METAMORPHIC LINK -->
+<xacro:property name="meta_cnt" value="3" />
+<xacro:property name="current_metalink" value="metalink_${meta_cnt}" />
+<xacro:property name="pseudo1_index" value="5" />
+<xacro:property name="pseudo2_index" value="6" />
 <!-- FINISHED 3RD METAMORPHIC LINK -->
 <!-- ADD 4TH ROBOT JOINT->SECOND DYNAMIXEL JOINT -> START -->
