Commit message: finished simplified xacro for 3rd metalink

File: xacros/conditioned_parameterized_SMM_assembly_6dof_for_ga.xacro (robot description, xacro)
@@ -96,5 +96,5 @@
 <xacro:property name="active_origin_rpy" value="${active['active_origin_rpy']}" />
 <!-- II.1	STRUCTURE STRING DEFINITION. This is imported by user  in the yaml file, based on desired structure/optimization results-->
-<xacro:property name="structure_string_definitions" value="/home/nikos/PhD/projects/Parametric_Simulation_Model_SMM/yamls/test/test_structure_string_definition_for_ga.yaml" />
+<xacro:property name="structure_string_definitions" value="/home/nikos/PhD/projects/Parametric_Simulation_Model_SMM/yamls/test/test_structure_string_definition_6dof_for_ga.yaml" />
 <xacro:property name="string_elements" value="${load_yaml(structure_string_definitions)}"/>
 <xacro:property name="s1" value="${string_elements['s1']}" /> <!-- Default: Active Joint 1 -->
@@ -242,5 +242,5 @@
 	<xacro:property name="active_cnt" value="1" />
 	<!-- MATLAB: Add active DXL: active_assembly_index = 2-->
-	<xacro:assembly_active_module2pseudo  active_assembly_name="${pseudo_b_name}_${pseudo_cnt}__${active_a_name}_${active_cnt}"  active_assembly_origin_rpy="${active2pseudo_origin_r} ${active2pseudo_origin_p_4_2} ${active2pseudo_origin_ry}" active_assembly_origin_xyz="${active2pseudo_origin_xyz}" active_assembly_parent="${pseudo_b_name}_${pseudo_cnt}" active_assembly_child="${active_a_name}_${active_cnt}" />
+	<xacro:assembly_active_module2pseudo  active_assembly_name="${pseudo_b_name}_${pseudo_cnt}__${active_a_name}_${active_cnt}"  active_assembly_origin_rpy="${active2pseudo_origin_r} ${active2pseudo_origin_p_10_2} ${active2pseudo_origin_ry}" active_assembly_origin_xyz="${active2pseudo_origin_xyz}" active_assembly_parent="${pseudo_b_name}_${pseudo_cnt}" active_assembly_child="${active_a_name}_${active_cnt}" />
 	<!-- Adds Active Module STATIC PART-->
 	<xacro:active_static_link_mesh name="${active_a_name}_${active_cnt}" origin_xyz="${active_a_origin_xyz}" origin_rpy="${active_a_origin_rpy}"/>
@@ -407,5 +407,5 @@
 	<xacro:property name="active_cnt" value="2" />
 	<!-- MATLAB: Add active DXL: active_assembly_index = 3-->
-	<xacro:assembly_active_module2pseudo  active_assembly_name="${pseudo_b_name}_${pseudo_cnt}__${active_a_name}_${active_cnt}"  active_assembly_origin_rpy="${active2pseudo_origin_r} ${active2pseudo_origin_p_4_3} ${active2pseudo_origin_ry}" active_assembly_origin_xyz="${active2pseudo_origin_xyz}" active_assembly_parent="${pseudo_b_name}_${pseudo_cnt}" active_assembly_child="${active_a_name}_${active_cnt}" />
+	<xacro:assembly_active_module2pseudo  active_assembly_name="${pseudo_b_name}_${pseudo_cnt}__${active_a_name}_${active_cnt}"  active_assembly_origin_rpy="${active2pseudo_origin_r} ${active2pseudo_origin_p_10_3} ${active2pseudo_origin_ry}" active_assembly_origin_xyz="${active2pseudo_origin_xyz}" active_assembly_parent="${pseudo_b_name}_${pseudo_cnt}" active_assembly_child="${active_a_name}_${active_cnt}" />
 	<!-- Adds Active Module STATIC PART-->
 	<xacro:active_static_link_mesh name="${active_a_name}_${active_cnt}" origin_xyz="${active_a_origin_xyz}" origin_rpy="${active_a_origin_rpy}"/>
@@ -414,12 +414,4 @@
 	<!-- Adds Active Module MOVING PART-->
 	<xacro:active_moving_link_mesh name="${active_b_name}_${active_cnt}" origin_xyz="${active_b_origin_xyz}" origin_rpy="${active_b_origin_rpy}"/>
-	<!-- Add TCP as TOOL frame-->
-	<!-- Add TCP -->
-	<joint name="${active_b_name}_${active_cnt}__TOOL" type="fixed">
-	    <origin rpy="0 0 0" xyz="0 0.05 0"/>
-	    <parent link="${active_b_name}_${active_cnt}"/>
-	    <child link="TOOL"/>
-	</joint>
-	<link name="TOOL"/>
 </xacro:if>
 <!-- ADD THIRD ROBOT JOINT->SECOND DYNAMIXEL JOINT -> END -->
@@ -437,6 +429,65 @@
 <xacro:property name="pseudo1_index" value="5" />
 <xacro:property name="pseudo2_index" value="6" />
+<xacro:unless value="${ s8 == 9}"> <!--  Case A is this meta link had pseudo in first string parameter => ONLY CASE BECAUSE IN GA THE FIRST PSEUDO MUST ALWAYS EXIST!-->
+		<xacro:property name="metalink_pseudo1" value="${current_metalink}_pseudo1" />
+		<xacro:if value="${ s8 == 31 }"> <!-- Case A.1.a -->
+			<xacro:synthetic_joint_name  synthetic_name="${active_b_name}_${active_cnt}__${metalink_pseudo1}_a"  synthetic_origin_rpy="${synthetic3_origin_r} ${synthetic_origin_xzp_4_p} ${synthetic3_origin_ry}" synthetic_origin_xyz="${synthetic_origin_xzp_4_x} ${synthetic3_origin_y} ${synthetic_origin_xzp_4_z}" synthetic_parent="${active_b_name}_${active_cnt}" synthetic_child="${metalink_pseudo1}_a" />
+			<!-- Start building Pseudojoint 2 STATIC PART-->
+			<xacro:pseudo_static_link_mesh name="${metalink_pseudo1}_a" origin_xyz="${pseudo_a_origin_xyz}" origin_rpy="${pseudo_a_origin_rpy}"/>
+			<!-- PSEUDO2 CONFIGURATION -->
+			<xacro:pseudo_joint_name  pseudo_name="${metalink_pseudo1}_a__${metalink_pseudo1}_b"  pseudo_origin_rpy="${pseudo_origin_r+pseudo5_angle} ${pseudo_origin_p} ${pseudo_origin_y}" pseudo_origin_xyz="${pseudo_origin_xyz}" pseudo_parent="${metalink_pseudo1}_a" pseudo_child="${metalink_pseudo1}_b" />
+			<!-- Start building Pseudojoint 2 MOVING PART-->
+			<xacro:pseudo_moving_link_mesh name="${metalink_pseudo1}_b" origin_xyz="${pseudo_b_origin_xyz}" origin_rpy="${pseudo_b_origin_rpy}"/>
+		</xacro:if>
+		<xacro:if value="${ s8 == 21}"> <!-- Case A.1.b -->
+			<xacro:synthetic_joint_name  synthetic_name="${active_b_name}_${active_cnt}__${metalink_pseudo1}_a"  synthetic_origin_rpy="${synthetic5_origin_r} ${synthetic_origin_xzp_4_p} ${synthetic5_origin_ry}" synthetic_origin_xyz="${synthetic_origin_xzp_4_x} ${synthetic5_origin_y} ${synthetic_origin_xzp_4_z}" synthetic_parent="${active_b_name}_${active_cnt}" synthetic_child="${metalink_pseudo1}_a" />
+			<!-- Start building Pseudojoint 2 STATIC PART-->
+			<xacro:pseudo_static_link_mesh name="${metalink_pseudo1}_a" origin_xyz="${pseudo_a_origin_xyz}" origin_rpy="${pseudo_a_origin_rpy}"/>
+			<!-- PSEUDO2 CONFIGURATION -->
+			<xacro:pseudo_joint_name  pseudo_name="${metalink_pseudo1}_a__${metalink_pseudo1}_b"  pseudo_origin_rpy="${pseudo_origin_r+pseudo5_angle} ${pseudo_origin_p} ${pseudo_origin_y}" pseudo_origin_xyz="${pseudo_origin_xyz}" pseudo_parent="${metalink_pseudo1}_a" pseudo_child="${metalink_pseudo1}_b" />
+			<!-- Start building Pseudojoint 2 MOVING PART-->
+			<xacro:pseudo_moving_link_mesh name="${metalink_pseudo1}_b" origin_xyz="${pseudo_b_origin_xyz}" origin_rpy="${pseudo_b_origin_rpy}"/>
+		</xacro:if>
+		<xacro:unless value="${ s9 == 9}"> <!-- Case A.1.c : and a 2nd pseudo exists-->
+			<xacro:property name="metalink_pseudo2" value="${current_metalink}_pseudo2" />
+			<xacro:if value="${ s9 == 21}"> <!-- Case A.1.c.1 -->
+				<xacro:synthetic_joint_name  synthetic_name="${metalink_pseudo1}_b__${metalink_pseudo2}_a"  synthetic_origin_rpy="${synthetic4_origin_r} ${synthetic_origin_xzp_5_p} ${synthetic4_origin_ry}" synthetic_origin_xyz="${synthetic_origin_xzp_5_x} ${synthetic4_origin_y} ${synthetic_origin_xzp_5_z}" synthetic_parent="${metalink_pseudo1}_b" synthetic_child="${metalink_pseudo2}_a" />
+				<!-- Start building Pseudojoint 2 STATIC PART-->
+				<xacro:pseudo_static_link_mesh name="${metalink_pseudo2}_a" origin_xyz="${pseudo_a_origin_xyz}" origin_rpy="${pseudo_a_origin_rpy}"/>
+				<!-- PSEUDO2 CONFIGURATION -->
+				<xacro:pseudo_joint_name  pseudo_name="${metalink_pseudo2}_a__${metalink_pseudo2}_b"  pseudo_origin_rpy="${pseudo_origin_r+pseudo5_angle} ${pseudo_origin_p} ${pseudo_origin_y}" pseudo_origin_xyz="${pseudo_origin_xyz}" pseudo_parent="${metalink_pseudo2}_a" pseudo_child="${metalink_pseudo2}_b" />
+				<!-- Start building Pseudojoint 2 MOVING PART-->
+				<xacro:pseudo_moving_link_mesh name="${metalink_pseudo2}_b" origin_xyz="${pseudo_b_origin_xyz}" origin_rpy="${pseudo_b_origin_rpy}"/>
+				<xacro:property name="last_body_assembled" value="${metalink_pseudo2}_b" />
+			</xacro:if>
+			<xacro:if value="${ s9 == 31}"> <!-- Case A.1.c.2 -->
+				<xacro:synthetic_joint_name  synthetic_name="${metalink_pseudo1}_b__${metalink_pseudo2}_a"  synthetic_origin_rpy="${synthetic2_origin_r} ${synthetic_origin_xzp_5_p} ${synthetic2_origin_ry}" synthetic_origin_xyz="${synthetic_origin_xzp_5_x} ${synthetic2_origin_y} ${synthetic_origin_xzp_5_z}" synthetic_parent="${metalink_pseudo1}_b" synthetic_child="${metalink_pseudo2}_a" />
+				<!-- Start building Pseudojoint 2 STATIC PART-->
+				<xacro:pseudo_static_link_mesh name="${metalink_pseudo2}_a" origin_xyz="${pseudo_a_origin_xyz}" origin_rpy="${pseudo_a_origin_rpy}"/>
+				<!-- PSEUDO2 CONFIGURATION -->
+				<xacro:pseudo_joint_name  pseudo_name="${metalink_pseudo2}_a__${metalink_pseudo2}_b"  pseudo_origin_rpy="${pseudo_origin_r+pseudo5_angle} ${pseudo_origin_p} ${pseudo_origin_y}" pseudo_origin_xyz="${pseudo_origin_xyz}" pseudo_parent="${metalink_pseudo2}_a" pseudo_child="${metalink_pseudo2}_b" />
+				<!-- Start building Pseudojoint 2 MOVING PART-->
+				<xacro:pseudo_moving_link_mesh name="${metalink_pseudo2}_b" origin_xyz="${pseudo_b_origin_xyz}" origin_rpy="${pseudo_b_origin_rpy}"/>
+				<xacro:property name="last_body_assembled" value="${metalink_pseudo2}_b" />
+			</xacro:if>
+		</xacro:unless>
+		<xacro:if value="${ s9 == 9}"> <!-- Case A.1.d : if a 2nd pseudo doesn't exist-->
+		// Add nothing here - only set naming connection with next active
+		<xacro:property name="last_body_assembled" value="${metalink_pseudo1}_b" />
+		</xacro:if>
+	</xacro:unless>	<!--  Case A - end-->
 <!-- FINISHED 3RD METAMORPHIC LINK -->
-<!-- ADD 4TH ROBOT JOINT->SECOND DYNAMIXEL JOINT -> START -->
+<!-- ADD 4TH ROBOT JOINT->3RD DYNAMIXEL JOINT -> START -->
+<xacro:if value="${s10 == 0}">
+	<xacro:property name="active_cnt" value="3" />
+	<!-- MATLAB: Add active DXL: active_assembly_index = 3-->
+	<xacro:assembly_active_module2pseudo  active_assembly_name="${last_body_assembled}__${active_a_name}_${active_cnt}"  active_assembly_origin_rpy="${active2pseudo_origin_r} ${active2pseudo_origin_p_11_1} ${active2pseudo_origin_ry}" active_assembly_origin_xyz="${active2pseudo_origin_xyz}" active_assembly_parent="${last_body_assembled}" active_assembly_child="${active_a_name}_${active_cnt}" />
+	<!-- Adds Active Module STATIC PART-->
+	<xacro:active_static_link_mesh name="${active_a_name}_${active_cnt}" origin_xyz="${active_a_origin_xyz}" origin_rpy="${active_a_origin_rpy}"/>
+	<!-- Adds DXL Active joint -->
+	<xacro:dxlPROp_joint active_name="${active_a_name}_${active_cnt}__${active_b_name}_${active_cnt}"  active_origin_rpy="${active_origin_rpy}" active_origin_xyz="${active_origin_xyz}" active_parent="${active_a_name}_${active_cnt}" active_child="${active_b_name}_${active_cnt}"/>
+	<!-- Adds Active Module MOVING PART-->
+	<xacro:active_moving_link_mesh name="${active_b_name}_${active_cnt}" origin_xyz="${active_b_origin_xyz}" origin_rpy="${active_b_origin_rpy}"/>
+</xacro:if>
 <!-- ADD 4TH ROBOT JOINT->SECOND DYNAMIXEL JOINT -> END -->
 <!-- STARTED 4TH METAMORPHIC LINK -->
@@ -448,3 +499,11 @@
 <!-- ADD 6TH ROBOT JOINT->SECOND DYNAMIXEL JOINT -> START -->
 <!-- ADD 6TH ROBOT JOINT->SECOND DYNAMIXEL JOINT -> END -->
+<!-- Add TCP as TOOL frame-->
+<!-- Add TCP -->
+<joint name="${active_b_name}_${active_cnt}__TOOL" type="fixed">
+    <origin rpy="0 0 0" xyz="0 0.05 0"/>
+    <parent link="${active_b_name}_${active_cnt}"/>
+    <child link="TOOL"/>
+</joint>
+<link name="TOOL"/>
 </robot>

File: xacros/metalink_cases_xacro_overview.xacro (robot description, xacro)
@@ -1,3 +1,5 @@
-<!-- STARTED METAMORPHIC LINK WITH PSEUDOS j & j+1 -->
+<!-- STARTED METAMORPHIC LINK WITH PSEUDOS j & j+1. These are the cases written for 3dof. For 6dof assembly a more
+     simplified version is implemented and can be found @ conditioned_parameterized_SMM_assembly_6dof_for_ga.xacro
+     @ Section "STARTED 3RD METAMORPHIC LINK" -->
 <xacro:unless value="${s_j == 9}"> <!--  Case A - start : this meta link had pseudo in first string parameter -->
 	<xacro:unless value="${s_j-1 == 9 or s_j-2 ==9}">  <!--  Case A.1 - start : {All} previous links had 2 pseudos-->

File: xacros/metalink_for_6dof_assembly.xacro (robot description, xacro)
@@ -4,12 +4,12 @@
      connectivity specified for passive modules of the metamorphic chain -->
 <!-- From overview: j-> pseudo_index -->
-<xacro:macro name="metalink_assembly" params="current_metalink pseudo1_string pseudo2_string">
+<xacro:macro name="metalink_assembly" params="current_metalink pseudo1_string pseudo2_string previous_body_name next_body_name synthetic_origin_xzp_metacnt_p synthetic_origin_xzp_metacnt_x synthetic_origin_xzp_metacnt_z">
 	<xacro:unless value="${ ${pseudo1_string} == 9}"> <!--  Case A is this meta link had pseudo in first string parameter => ONLY CASE BECAUSE IN GA THE FIRST PSEUDO MUST ALWAYS EXIST!-->
 		<xacro:property name="metalink_pseudo1" value="${current_metalink}_pseudo1" />
 		<xacro:if value="${ ${pseudo1_string} == 31 }"> <!-- Case A.1.a -->
 			<!-- naming must change! -->
-			<xacro:synthetic_joint_name  synthetic_name="${pseudo_b_name}_${last_pseudo_cnt}__${pseudo_a_name}_${pseudo_cnt}"  synthetic_origin_rpy="${synthetic2_origin_r} ${synthetic_origin_xzp_3_p} ${synthetic2_origin_ry}" synthetic_origin_xyz="${synthetic_origin_xzp_3_x} ${synthetic2_origin_y} ${synthetic_origin_xzp_3_z}" synthetic_parent="${pseudo_b_name}_${last_pseudo_cnt}" synthetic_child="${pseudo_a_name}_${pseudo_cnt}" />
+			<xacro:synthetic_joint_name  synthetic_name="${previous_body_name}__${metalink_pseudo1}_1"  synthetic_origin_rpy="${synthetic2_origin_r} ${synthetic_origin_xzp_metacnt_p} ${synthetic2_origin_ry}" synthetic_origin_xyz="${synthetic_origin_xzp_metacnt_x} ${synthetic2_origin_y} ${synthetic_origin_xzp_metacnt_z}" synthetic_parent="${previous_body_name}" synthetic_child="${metalink_pseudo1}_1" />
 			<!-- Start building Pseudojoint 2 STATIC PART-->
-			<xacro:pseudo_static_link_mesh name="${pseudo_a_name}_${pseudo_cnt}" origin_xyz="${pseudo_a_origin_xyz}" origin_rpy="${pseudo_a_origin_rpy}"/>
+			<xacro:pseudo_static_link_mesh name="${metalink_pseudo1}_1" origin_xyz="${pseudo_a_origin_xyz}" origin_rpy="${pseudo_a_origin_rpy}"/>
 			<!-- PSEUDO2 CONFIGURATION -->
 			<xacro:pseudo_joint_name  pseudo_name="${pseudo_a_name}_${pseudo_cnt}__${pseudo_b_name}_${pseudo_cnt}"  pseudo_origin_rpy="${pseudo_origin_r+pseudo4_angle} ${pseudo_origin_p} ${pseudo_origin_y}" pseudo_origin_xyz="${pseudo_origin_xyz}" pseudo_parent="${pseudo_a_name}_${pseudo_cnt}" pseudo_child="${pseudo_b_name}_${pseudo_cnt}" />
