Commit message: just visualization of extracted TSP results

File: xacros/conditioned_parameterized_SMM_assembly_6dof_for_ga2.xacro (robot description, xacro)
@@ -64,13 +64,13 @@
 <xacro:property name="last_pseudo_cnt" value="0" />
 <!--
-<xacro:property name="pseudo1_angle" value="1.5708"/>
-<xacro:property name="pseudo2_angle" value="0.5"/>
-<xacro:property name="pseudo3_angle" value="0"/>
-<xacro:property name="pseudo4_angle" value="0.7854"/>
+<xacro:property name="pseudo1_angle" value="-1.5708"/>
+<xacro:property name="pseudo2_angle" value="-0.5"/>
+<xacro:property name="pseudo3_angle" value="0.7854"/>
+<xacro:property name="pseudo4_angle" value="-1"/>
 <xacro:property name="pseudo5_angle" value="-0.7854"/>
-<xacro:property name="pseudo6_angle" value="0"/>
-<xacro:property name="pseudo7_angle" value="0"/>
+<xacro:property name="pseudo6_angle" value="1.15"/>
+<xacro:property name="pseudo7_angle" value="0.85"/>
 <xacro:property name="pseudo8_angle" value="1.5708"/>
-<xacro:property name="pseudo9_angle" value="0"/>
+<xacro:property name="pseudo9_angle" value="-0.45"/>
 <xacro:property name="pseudo10_angle" value="-1.5708"/>
 -->

File: xacros/conditioned_parameterized_SMM_assembly_for_ga2.xacro (robot description, xacro)
@@ -66,8 +66,15 @@
 <xacro:property name="pseudo_cnt" value="0" />
 <xacro:property name="last_pseudo_cnt" value="0" />
+<!--MATLAB pseudoangle calculation: deg2rad(15) * (floor(ci)-1) + (-1.5708)-->
+<!--
 <xacro:property name="pseudo1_angle" value="0"/>
 <xacro:property name="pseudo2_angle" value="0"/>
 <xacro:property name="pseudo3_angle" value="0"/>
 <xacro:property name="pseudo4_angle" value="0"/>
+-->
+<xacro:property name="pseudo1_angle" value="-1.3464"/>
+<xacro:property name="pseudo2_angle" value="-0.8976"/>
+<xacro:property name="pseudo3_angle" value="0.4488"/>
+<xacro:property name="pseudo4_angle" value="-1.3464"/>
 <!-- ACTIVE2PSEUDOS FIXED TFs -->
 <xacro:property name="active2pseudo" value="${load_yaml(definitions_file)}"/>

File: xacros/generated_urdf_from_xacros_here/test_3dof.urdf (robot description, URDF)
Before this commit: robot ovidius_smm, 14 links, 13 joints
Joints:
- joint active_module_b_1__metalink_2_pseudo1_a: origin xyz=0.001 0.0955 -0.025 rpy=0 -1.5708 0 -> xyz=0.001 0.0525 -0.055 rpy=-1.5708 -1.5708 0
- joint metalink_1_pseudo1_a__metalink_1_pseudo1_b: origin xyz=0 0.025 0.118 rpy=1.5708 0 0 -> xyz=0 0.025 0.118 rpy=3.1416 0 0
- joint metalink_1_pseudo1_b__metalink_1_pseudo2_a: origin xyz=0 0.1444 0.03 rpy=0 0.7854 0 -> xyz=-0.005 0.1444 0.005 rpy=0 0.78 0
- joint metalink_1_pseudo2_a__metalink_1_pseudo2_b: origin xyz=0 0.025 0.118 rpy=1.5708 0 0 -> xyz=0 0.025 0.118 rpy=0.7854 0 0
- joint metalink_2_pseudo1_a__metalink_2_pseudo1_b: origin xyz=0 0.025 0.118 rpy=1.5708 0 0 -> xyz=0 0.025 0.118 rpy=3.1416 0 0
- joint metalink_2_pseudo1_b__metalink_2_pseudo2_a: origin xyz=0.005 0.101 -0.003 rpy=-1.5708 -1.5708 0 -> xyz=0.003 0.1444 -0.001 rpy=0 1.5708 0
- joint metalink_2_pseudo2_a__metalink_2_pseudo2_b: origin xyz=0 0.025 0.118 rpy=1.5708 0 0 -> xyz=0 0.025 0.118 rpy=2.3562 0 0
- joint metalink_2_pseudo2_b__active_module_a_2: origin xyz=0 0.1 0 rpy=0 1.5708 0 -> xyz=0 0.1 0 rpy=0 0 0

File: xacros/generated_urdf_from_xacros_here/test_3dof_ref_anat.urdf (robot description, URDF)
Before this commit: robot ovidius_smm, 10 links, 9 joints
Joints:
- joint metalink_1_pseudo1_a__metalink_1_pseudo1_b: origin xyz=0 0.025 0.118 rpy=2.3562 0 0 -> xyz=0 0.025 0.118 rpy=1.5708 0 0
- joint metalink_2_pseudo1_a__metalink_2_pseudo1_b: origin xyz=0 0.025 0.118 rpy=0.0 0 0 -> xyz=0 0.025 0.118 rpy=1.5708 0 0

File: xacros/generated_urdf_from_xacros_here/test_6dof_ref_anat.urdf (robot description, URDF)
Before this commit: robot ovidius_smm_6DoF, 31 links, 30 joints
Links:
- removed link metalink_2_pseudo2_a
- removed link metalink_2_pseudo2_b
Joints:
- removed joint metalink_2_pseudo1_b__metalink_2_pseudo2_a
- removed joint metalink_2_pseudo2_a__metalink_2_pseudo2_b
- removed joint metalink_2_pseudo2_b__active_module_a_2
- added joint metalink_2_pseudo1_b__active_module_a_2: type fixed, parent metalink_2_pseudo1_b, child active_module_a_2, origin xyz=0 0.1 0 rpy=0 0 0
- joint active_module_b_1__metalink_2_pseudo1_a: origin xyz=-0.035 0.0525 0 rpy=-1.5708 1.5708 0 -> xyz=-0.035 0.0525 0.005 rpy=-1.5708 1.5708 0
- joint active_module_b_2__metalink_3_pseudo1_a: origin xyz=-0.0058 0.0955 0 rpy=0 0 0 -> xyz=0.0058 0.0955 0 rpy=0 0.7854 0
- joint active_module_b_4__metalink_5_pseudo1_a: origin xyz=0.05 0.0525 0 rpy=-1.5708 -1.5708 0 -> xyz=-0.05 0.0525 0 rpy=-1.5708 1.5708 0
- joint metalink_3_pseudo1_b__metalink_3_pseudo2_a: origin xyz=0 0.101 0 rpy=-1.5708 -1.5708 0 -> xyz=0 0.1444 0 rpy=0 -1.5708 0
- joint metalink_5_pseudo1_b__metalink_5_pseudo2_a: origin xyz=0 0.101 0.005 rpy=-1.5708 -0.7854 0 -> xyz=0 0.1444 0 rpy=0 0.7854 0
- joint metalink_5_pseudo2_b__active_module_a_5: origin xyz=0 0.1 0 rpy=0 1.5708 0 -> xyz=0 0.1 0 rpy=0 0 0

File: xacros/generated_urdf_from_xacros_here/test_6dof_test_anat.urdf (robot description, URDF)
Before this commit: robot ovidius_smm_6DoF, 31 links, 30 joints
Links:
- removed link metalink_2_pseudo2_a
- removed link metalink_2_pseudo2_b
Joints:
- removed joint metalink_2_pseudo1_b__metalink_2_pseudo2_a
- removed joint metalink_2_pseudo2_a__metalink_2_pseudo2_b
- removed joint metalink_2_pseudo2_b__active_module_a_2
- added joint metalink_2_pseudo1_b__active_module_a_2: type fixed, parent metalink_2_pseudo1_b, child active_module_a_2, origin xyz=0 0.1 0 rpy=0 0 0
- joint active_module_b_1__metalink_2_pseudo1_a: origin xyz=-0.035 0.0525 0 rpy=-1.5708 1.5708 0 -> xyz=-0.035 0.0525 0.005 rpy=-1.5708 1.5708 0
- joint active_module_b_2__metalink_3_pseudo1_a: origin xyz=-0.0058 0.0955 0 rpy=0 0 0 -> xyz=0.0058 0.0955 0 rpy=0 0.7854 0
- joint active_module_b_4__metalink_5_pseudo1_a: origin xyz=0.05 0.0525 0 rpy=-1.5708 -1.5708 0 -> xyz=-0.05 0.0525 0 rpy=-1.5708 1.5708 0
- joint metalink_1_pseudo1_a__metalink_1_pseudo1_b: origin xyz=0 0.025 0.118 rpy=3.1416 0 0 -> xyz=0 0.025 0.118 rpy=0.0 0 0
- joint metalink_2_pseudo1_a__metalink_2_pseudo1_b: origin xyz=0 0.025 0.118 rpy=1.5708 0 0 -> xyz=0 0.025 0.118 rpy=2.3562 0 0
- joint metalink_3_pseudo1_b__metalink_3_pseudo2_a: origin xyz=0 0.101 0 rpy=-1.5708 -1.5708 0 -> xyz=0 0.1444 0 rpy=0 -1.5708 0
- joint metalink_3_pseudo2_a__metalink_3_pseudo2_b: origin xyz=0 0.025 0.118 rpy=1.5708 0 0 -> xyz=0 0.025 0.118 rpy=2.7208 0 0
- joint metalink_4_pseudo1_a__metalink_4_pseudo1_b: origin xyz=0 0.025 0.118 rpy=1.5708 0 0 -> xyz=0 0.025 0.118 rpy=2.4208 0 0
- joint metalink_5_pseudo1_a__metalink_5_pseudo1_b: origin xyz=0 0.025 0.118 rpy=1.5708 0 0 -> xyz=0 0.025 0.118 rpy=1.1208 0 0
- joint metalink_5_pseudo1_b__metalink_5_pseudo2_a: origin xyz=0 0.101 0.005 rpy=-1.5708 -0.7854 0 -> xyz=0 0.1444 0 rpy=0 0.7854 0
- joint metalink_5_pseudo2_b__active_module_a_5: origin xyz=0 0.1 0 rpy=0 1.5708 0 -> xyz=0 0.1 0 rpy=0 0 0
