Commit message: sync from laptop because of error-msg

File: xacros/conditioned_parameterized_SMM_assembly_for_ga2.xacro (robot description, xacro)
@@ -66,7 +66,14 @@
 <xacro:property name="pseudo_cnt" value="0" />
 <xacro:property name="last_pseudo_cnt" value="0" />
+<!--MATLAB pseudoangle calculation: deg2rad(15) * (floor(ci)-1) + (-1.5708)-->
+<!--
 <xacro:property name="pseudo1_angle" value="0"/>
 <xacro:property name="pseudo2_angle" value="0"/>
 <xacro:property name="pseudo3_angle" value="0"/>
+<xacro:property name="pseudo4_angle" value="0"/>
+-->
+<xacro:property name="pseudo1_angle" value="0.2618"/>
+<xacro:property name="pseudo2_angle" value="0.2618"/>
+<xacro:property name="pseudo3_angle" value="-0.5236"/>
 <xacro:property name="pseudo4_angle" value="0"/>
 <!-- ACTIVE2PSEUDOS FIXED TFs -->

Commit message: LAPTOP-added pseudo yaml

File: xacros/conditioned_parameterized_SMM_assembly_for_ga2.xacro (robot description, xacro)
@@ -67,5 +67,5 @@
 <xacro:property name="last_pseudo_cnt" value="0" />
 <!--MATLAB pseudoangle calculation: deg2rad(15) * (floor(ci)-1) + (-1.5708)-->
-<!--
+<!-- Only for Reference anatomy -> Deprecated[8-4-21]
 <xacro:property name="pseudo1_angle" value="0"/>
 <xacro:property name="pseudo2_angle" value="0"/>
@@ -73,19 +73,16 @@
 <xacro:property name="pseudo4_angle" value="0"/>
 -->
-<<<<<<< HEAD
-<!-- These should be passed to a yaml file -->
-=======
-<<<<<<< HEAD
+<!-- These should be passed to a yaml file
 <xacro:property name="pseudo1_angle" value="0.2618"/>
 <xacro:property name="pseudo2_angle" value="0.2618"/>
 <xacro:property name="pseudo3_angle" value="-0.5236"/>
-<xacro:property name="pseudo4_angle" value="0"/>
-=======
->>>>>>> 25c8464eea53b0f6d06c1b83d260fc1826c44131
-<xacro:property name="pseudo1_angle" value="-1.3464"/>
-<xacro:property name="pseudo2_angle" value="-0.8976"/>
-<xacro:property name="pseudo3_angle" value="0.4488"/>
-<xacro:property name="pseudo4_angle" value="-1.3464"/>
->>>>>>> fbe4a2184dda8047b0cf65f0641a40f554687589
+<xacro:property name="pseudo4_angle" value="0"/> -->
+<!-- [8-4-21] Passed from a yaml file -->
+<xacro:property name="pseudo_angles_definitions" value="/home/nikos/PhD/projects/Parametric_Simulation_Model_SMM/yamls/test/pseudo_angles_for_ovidius_robot_for_ga.yaml" />
+<xacro:property name="pseudo_angles" value="${load_yaml(pseudo_angles_definitions)}"/>
+<xacro:property name="pseudo1_angle" value="${pseudo_angles['pseudo1_angle']}" />
+<xacro:property name="pseudo2_angle" value="${pseudo_angles['pseudo2_angle']}" />
+<xacro:property name="pseudo3_angle" value="${pseudo_angles['pseudo3_angle']}" />
+<xacro:property name="pseudo4_angle" value="${pseudo_angles['pseudo4_angle']}" />
 <!-- ACTIVE2PSEUDOS FIXED TFs -->
 <xacro:property name="active2pseudo" value="${load_yaml(definitions_file)}"/>
